File: PCB Layouts/Layout 2_15/Selection Interface.sch (KiCad schematic (older format))
At the start: 127 parts, among them P1 CONN_01X02, P11 CONN_01X02, P12 CONN_01X02, P13 CONN_01X10, P14 CONN_01X02, P15 CONN_01X02, P16 CONN_01X02, P18 CONN_02X05, P19 CONN_02X05, P2 CONN_01X02, P21 CONN_02X05, P3 CONN_01X02, P4 CONN_01X02, P5 CONN_01X02, P6 CONN_02X10, P7 CONN_01X02, P8 CONN_02X04, P9 CONN_01X02, U1 CY8C42_(48_TQFP), U2 CY8C42_(48_TQFP), U3 CY8C58_(100_TQFP), U4 CY8C42_(48_TQFP), U5 68_PLCC_Socket_(8468-21B1-RK-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, U6 CY8C42_(48_TQFP), U7 CY8C58_(100_TQFP), U8 USB_2.0_B, U9 USB_2.0_B

Commit message: Updated the footprints in Layout 2_15 to be from the newest standard libraries
Parts:
- C1, C10, C11, C12, C13, C14, C15, C16, C17, C18, C19, C2, C20, C21, C22, C23, C24, C25, C26, C27, C28, C29, C3, C30, C31, C32, C33, C34, C35, C36, C37, C38, C39, C4, C40, C41, C42, C43, C44, C45, C46, C47, C48, C49, C5, C50, C51, C52, C53, C54, C55, C56, C57, C58, C59, C6, C60, C61, C62, C63, C64, C65, C66, C67, C68, C69, C7, C70, C71, C72, C73, C74, C8, C9: footprint Capacitors_SMD:C_0603 -> Capacitor_SMD:C_0603_1608Metric
- FB1, FB2, FB3, FB4, FB5, FB6, FB7, FB8, R1, R10, R11, R12, R13, R14, R15, R16, R17, R18, R2, R3, R4, R5, R6, R7, R8, R9: footprint Resistors_SMD:R_0603 -> Resistor_SMD:R_0603_1608Metric
- P13: footprint NoyceLibrary:Headers_SMD_1x10_(cut_95157-240LF) -> Connector_PinHeader_2.54mm:PinHeader_1x10_P2.54mm_Vertical_SMD_Pin1Left
- P18, P19, P21: footprint NoyceLibrary:Headers_SMD_2x5_(cut_95157-240LF) -> Connector_PinHeader_2.54mm:PinHeader_2x05_P2.54mm_Vertical_SMD
- P6: footprint NoyceLibrary:Headers_SMD_2x10_(cut_95157-240LF) -> Connector_PinHeader_2.54mm:PinHeader_2x10_P2.54mm_Vertical_SMD
- P8: footprint NoyceLibrary:Headers_SMD_2x4_(cut_95157-240LF) -> Connector_PinHeader_2.54mm:PinHeader_2x04_P2.54mm_Vertical_SMD
- U1, U2, U4, U6: footprint Housings_QFP:TQFP-48_7x7mm_Pitch0.5mm -> Package_QFP:TQFP-48_7x7mm_P0.5mm
- U3, U7: footprint Housings_QFP:TQFP-100_14x14mm_Pitch0.5mm -> Package_QFP:TQFP-100_14x14mm_P0.5mm
- U8: footprint NoyceLibrary:Micro_USB_2.0_B_SMD(10118192-0001LF) -> Connector_USB:USB_Micro-B_Amphenol_10103594-0001LF_Horizontal

Commit message: Added a project-specific custom footprint library that contains anything not found in standard libraries
Parts:
- P1, P11, P12, P14, P15, P16, P2, P3, P4, P5, P7, P9: footprint NoyceLibrary:IPEX_Connector_SMD_(RECE.20279.001E.01) -> Custom_Footprint_Library:IPEX_Connector_SMD_(RECE.20279.001E.01)
- U5: footprint NoyceLibrary:68_PLCC_Socket_(8468-21B1-RK-TP) -> Custom_Footprint_Library:68_PLCC_Socket_(8468-21B1-RK-TP)
- U8: footprint Connector_USB:USB_Micro-B_Amphenol_10103594-0001LF_Horizontal -> Custom_Footprint_Library:Micro_USB_2.0_B_SMD(10118192-0001LF)
- U9: footprint NoyceLibrary:Micro_USB_2.0_B_SMD(10118192-0001LF) -> Custom_Footprint_Library:Micro_USB_2.0_B_SMD(10118192-0001LF)
Changed lines of the file:
@@
 F 0 "U5" H 1900 4050 50  0000 C CNN
 F 1 "68_PLCC_Socket_(8468-21B1-RK-TP)" H 1900 4250 50  0000 C CNN
-F 2 "NoyceLibrary:68_PLCC_Socket_(8468-21B1-RK-TP)" H 1900 4150 50  0001 C CNN
+F 2 "Custom_Footprint_Library:68_PLCC_Socket_(8468-21B1-RK-TP)" H 1900 4150 50  0001 C CNN
 F 3 "DOCUMENTATION" H 1900 4150 50  0001 C CNN
 	1    1900 4150
@@
 F 0 "P4" H 4250 6150 50  0000 C CNN
 F 1 "CONN_01X02" V 4350 6000 50  0000 C CNN
-F 2 "NoyceLibrary:IPEX_Connector_SMD_(RECE.20279.001E.01)" H 4250 6000 50  0001 C CNN
+F 2 "Custom_Footprint_Library:IPEX_Connector_SMD_(RECE.20279.001E.01)" H 4250 6000 50  0001 C CNN
 F 3 "" H 4250 6000 50  0000 C CNN
 	1    4250 6000
@@
 F 0 "P3" H 3750 6150 50  0000 C CNN
 F 1 "CONN_01X02" V 3850 6000 50  0000 C CNN
-F 2 "NoyceLibrary:IPEX_Connector_SMD_(RECE.20279.001E.01)" H 3750 6000 50  0001 C CNN
+F 2 "Custom_Footprint_Library:IPEX_Connector_SMD_(RECE.20279.001E.01)" H 3750 6000 50  0001 C CNN
 F 3 "" H 3750 6000 50  0000 C CNN
 	1    3750 6000
@@
 F 0 "P2" H 3250 6150 50  0000 C CNN
 F 1 "CONN_01X02" V 3350 6000 50  0000 C CNN
-F 2 "NoyceLibrary:IPEX_Connector_SMD_(RECE.20279.001E.01)" H 3250 6000 50  0001 C CNN
+F 2 "Custom_Footprint_Library:IPEX_Connector_SMD_(RECE.20279.001E.01)" H 3250 6000 50  0001 C CNN
 F 3 "" H 3250 6000 50  0000 C CNN
 	1    3250 6000
@@
 F 0 "P1" H 2750 6150 50  0000 C CNN
 F 1 "CONN_01X02" V 2850 6000 50  0000 C CNN
-F 2 "NoyceLibrary:IPEX_Connector_SMD_(RECE.20279.001E.01)" H 2750 6000 50  0001 C CNN
+F 2 "Custom_Footprint_Library:IPEX_Connector_SMD_(RECE.20279.001E.01)" H 2750 6000 50  0001 C CNN
 F 3 "" H 2750 6000 50  0000 C CNN
 	1    2750 6000
@@
 F 0 "P5" H 4750 6150 50  0000 C CNN
 F 1 "CONN_01X02" V 4850 6000 50  0000 C CNN
-F 2 "NoyceLibrary:IPEX_Connector_SMD_(RECE.20279.001E.01)" H 4750 6000 50  0001 C CNN
+F 2 "Custom_Footprint_Library:IPEX_Connector_SMD_(RECE.20279.001E.01)" H 4750 6000 50  0001 C CNN
 F 3 "" H 4750 6000 50  0000 C CNN
 	1    4750 6000
@@
 F 0 "P7" H 5250 6150 50  0000 C CNN
 F 1 "CONN_01X02" V 5350 6000 50  0000 C CNN
-F 2 "NoyceLibrary:IPEX_Connector_SMD_(RECE.20279.001E.01)" H 5250 6000 50  0001 C CNN
+F 2 "Custom_Footprint_Library:IPEX_Connector_SMD_(RECE.20279.001E.01)" H 5250 6000 50  0001 C CNN
 F 3 "" H 5250 6000 50  0000 C CNN
 	1    5250 6000
@@
 F 0 "P9" H 5750 6150 50  0000 C CNN
 F 1 "CONN_01X02" V 5850 6000 50  0000 C CNN
-F 2 "NoyceLibrary:IPEX_Connector_SMD_(RECE.20279.001E.01)" H 5750 6000 50  0001 C CNN
+F 2 "Custom_Footprint_Library:IPEX_Connector_SMD_(RECE.20279.001E.01)" H 5750 6000 50  0001 C CNN
 F 3 "" H 5750 6000 50  0000 C CNN
 	1    5750 6000
@@
 F 0 "P15" H 7750 6150 50  0000 C CNN
 F 1 "CONN_01X02" V 7850 6000 50  0000 C CNN
-F 2 "NoyceLibrary:IPEX_Connector_SMD_(RECE.20279.001E.01)" H 7750 6000 50  0001 C CNN
+F 2 "Custom_Footprint_Library:IPEX_Connector_SMD_(RECE.20279.001E.01)" H 7750 6000 50  0001 C CNN
 F 3 "" H 7750 6000 50  0000 C CNN
 	1    7750 6000
@@
 F 0 "P14" H 7250 6150 50  0000 C CNN
 F 1 "CONN_01X02" V 7350 6000 50  0000 C CNN
-F 2 "NoyceLibrary:IPEX_Connector_SMD_(RECE.20279.001E.01)" H 7250 6000 50  0001 C CNN
+F 2 "Custom_Footprint_Library:IPEX_Connector_SMD_(RECE.20279.001E.01)" H 7250 6000 50  0001 C CNN
 F 3 "" H 7250 6000 50  0000 C CNN
 	1    7250 6000
@@
 F 0 "P12" H 6750 6150 50  0000 C CNN
 F 1 "CONN_01X02" V 6850 6000 50  0000 C CNN
-F 2 "NoyceLibrary:IPEX_Connector_SMD_(RECE.20279.001E.01)" H 6750 6000 50  0001 C CNN
+F 2 "Custom_Footprint_Library:IPEX_Connector_SMD_(RECE.20279.001E.01)" H 6750 6000 50  0001 C CNN
 F 3 "" H 6750 6000 50  0000 C CNN
 	1    6750 6000
@@
 F 0 "P11" H 6250 6150 50  0000 C CNN
 F 1 "CONN_01X02" V 6350 6000 50  0000 C CNN
-F 2 "NoyceLibrary:IPEX_Connector_SMD_(RECE.20279.001E.01)" H 6250 6000 50  0001 C CNN
+F 2 "Custom_Footprint_Library:IPEX_Connector_SMD_(RECE.20279.001E.01)" H 6250 6000 50  0001 C CNN
 F 3 "" H 6250 6000 50  0000 C CNN
 	1    6250 6000
@@
 F 0 "P16" H 8250 6150 50  0000 C CNN
 F 1 "CONN_01X02" V 8350 6000 50  0000 C CNN
-F 2 "NoyceLibrary:IPEX_Connector_SMD_(RECE.20279.001E.01)" H 8250 6000 50  0001 C CNN
+F 2 "Custom_Footprint_Library:IPEX_Connector_SMD_(RECE.20279.001E.01)" H 8250 6000 50  0001 C CNN
 F 3 "" H 8250 6000 50  0000 C CNN
 	1    8250 6000
@@
 F 0 "U8" H 17300 5700 60  0000 C CNN
 F 1 "USB_2.0_B" H 17300 5600 60  0000 C CNN
-F 2 "Connector_USB:USB_Micro-B_Amphenol_10103594-0001LF_Horizontal" H 17300 5650 60  0001 C CNN
+F 2 "Custom_Footprint_Library:Micro_USB_2.0_B_SMD(10118192-0001LF)" H 17300 5650 60  0001 C CNN
 F 3 "" H 17300 5650 60  0001 C CNN
 	1    17300 5650
@@
 F 0 "U9" H 26450 5900 60  0000 C CNN
 F 1 "USB_2.0_B" H 26450 5800 60  0000 C CNN
-F 2 "NoyceLibrary:Micro_USB_2.0_B_SMD(10118192-0001LF)" H 26450 5850 60  0001 C CNN
+F 2 "Custom_Footprint_Library:Micro_USB_2.0_B_SMD(10118192-0001LF)" H 26450 5850 60  0001 C CNN
 F 3 "" H 26450 5850 60  0001 C CNN
 	1    26450 5850

Commit message: Regenerated and loaded the netlist for Layout 2_15. All components are now switched over to the most up-to-date footprints. Added mounting holes to the schematic and layout. The design is now ready for a more significant overhaul, so will likely be creating a new version soon.
Parts:
- added MH1, MH2, MH3, MH5, MH6: MountingHole, Custom_Footprint_Library:MountingHole_5.1mm, symbol Mechanical:MountingHole
Changed lines of the file:
@@
 Wire Wire Line
 	4400 2200 4400 2300
+$Comp
+L Mechanical:MountingHole MH3
+U 1 1 5D9EABCE
+P 10100 5250
+F 0 "MH3" H 10200 5296 50  0000 L CNN
+F 1 "MountingHole" H 10200 5205 50  0000 L CNN
+F 2 "Custom_Footprint_Library:MountingHole_5.1mm" H 10100 5250 50  0001 C CNN
+F 3 "~" H 10100 5250 50  0001 C CNN
+	1    10100 5250
+	1    0    0    -1
+$EndComp
+$Comp
+L Mechanical:MountingHole MH2
+U 1 1 5D9EBACA
+P 10100 5000
+F 0 "MH2" H 10200 5046 50  0000 L CNN
+F 1 "MountingHole" H 10200 4955 50  0000 L CNN
+F 2 "Custom_Footprint_Library:MountingHole_5.1mm" H 10100 5000 50  0001 C CNN
+F 3 "~" H 10100 5000 50  0001 C CNN
+	1    10100 5000
+	1    0    0    -1
+$EndComp
+$Comp
+L Mechanical:MountingHole MH5
+U 1 1 5DA59D68
+P 10100 5750
+F 0 "MH5" H 10200 5796 50  0000 L CNN
+F 1 "MountingHole" H 10200 5705 50  0000 L CNN
+F 2 "Custom_Footprint_Library:MountingHole_5.1mm" H 10100 5750 50  0001 C CNN
+F 3 "~" H 10100 5750 50  0001 C CNN
+	1    10100 5750
+	1    0    0    -1
+$EndComp
+$Comp
+L Mechanical:MountingHole MH6
+U 1 1 5DA59F0E
+P 10100 6000
+F 0 "MH6" H 10200 6046 50  0000 L CNN
+F 1 "MountingHole" H 10200 5955 50  0000 L CNN
+F 2 "Custom_Footprint_Library:MountingHole_5.1mm" H 10100 6000 50  0001 C CNN
+F 3 "~" H 10100 6000 50  0001 C CNN
+	1    10100 6000
+	1    0    0    -1
+$EndComp
+$Comp
+L Mechanical:MountingHole MH1
+U 1 1 5DA5A0AE
+P 10100 4750
+F 0 "MH1" H 10200 4796 50  0000 L CNN
+F 1 "MountingHole" H 10200 4705 50  0000 L CNN
+F 2 "Custom_Footprint_Library:MountingHole_5.1mm" H 10100 4750 50  0001 C CNN
+F 3 "~" H 10100 4750 50  0001 C CNN
+	1    10100 4750
+	1    0    0    -1
+$EndComp
 $EndSCHEMATC

Commit message: Fixed swapping of Back gate and solution gate in Layout 2_15
Other:
- note added: "- Don’t have gates permanently connected to PSoCs\n- Break out I2C\n- Give Masters ability to reset Slaves\n- Add more optional TIA resistors\n- Give PSoCs more natural number labels\n- Communication between Masters\n- Clock sync between Masters\n- Resistor dividers for input measurements (esp. from AFM)\n- Boost converter for larger gate drive on board\n- Add interface for external chip (tire se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"
- note removed: "- Don't have gates permanently connected to PSoCs\n- Break out I2C\n- Give Masters ability to reset Slaves\n- Add more optional TIA resistors\n- Give PSoCs more natural number labels\n- Communication between Masters\n- Clock sync between Masters\n- Resistor dividers for input measurements (esp. from AFM)\n- Boost converter for larger gate drive on board\n- Add interface for external chip (tire se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"
Changed lines of the file:
@@
 LocalGates
 Text GLabel 1150 900  0    39   Input ~ 0
+SolutionGate
+Text GLabel 1150 1000 0    39   Input ~ 0
 BackGate
-Text GLabel 1150 1000 0    39   Input ~ 0
-SolutionGate
 Text GLabel 1150 1200 0    60   Input ~ 0
 D1
@@
 GND
 Text GLabel 3900 1700 0    39   Input ~ 0
+BackGate
+Text GLabel 3900 1500 0    39   Input ~ 0
 SolutionGate
-Text GLabel 3900 1500 0    39   Input ~ 0
-BackGate
 Text GLabel 3050 3100 0    39   Input ~ 0
 I1
@@
 GND
 Text GLabel 3150 3200 2    39   Input ~ 0
-BackGate
+SolutionGate
 Text GLabel 3150 3300 2    39   Input ~ 0
 LocalGates
 Text GLabel 3150 3400 2    39   Input ~ 0
-SolutionGate
+BackGate
 Text GLabel 3150 3600 2    39   Input ~ 0
 S2
@@
 I1
 Text GLabel 3300 5800 1    39   Input ~ 0
-I2
+SolutionGate
 Text GLabel 3800 5800 1    39   Input ~ 0
-I3
+LocalGates
 Text GLabel 4300 5800 1    39   Input ~ 0
-I4
+BackGate
 Text GLabel 4800 5800 1    39   Input ~ 0
-I5
+S1
 Text GLabel 5300 5800 1    39   Input ~ 0
-I6
+S2
 Text GLabel 5800 5800 1    39   Input ~ 0
-I7
+S3
 Text GLabel 6300 5800 1    39   Input ~ 0
-I8
+S4
 Text GLabel 6800 5800 1    39   Input ~ 0
 I9
@@
 	5600 3700 5150 3700
 Text Notes 6600 3750 0    60   ~ 0
-- Don't have gates permanently connected to PSoCs\n- Break out I2C\n- Give Masters ability to reset Slaves\n- Add more optional TIA resistors\n- Give PSoCs more natural number labels\n- Communication between Masters\n- Clock sync between Masters\n- Resistor dividers for input measurements (esp. from AFM)\n- Boost converter for larger gate drive on board\n- Add interface for external chip (tire sensors)\n- Add interface for non-packaged chip (pogo pins)\n- Add temperature, humidity, and pressure sensors\n- Solution Gate and Back Gate are switched on Socket!  Fix!\n- Need holes for magnets or something to preserve absolute positioning on AFM stage\n
+- Don’t have gates permanently connected to PSoCs\n- Break out I2C\n- Give Masters ability to reset Slaves\n- Add more optional TIA resistors\n- Give PSoCs more natural number labels\n- Communication between Masters\n- Clock sync between Masters\n- Resistor dividers for input measurements (esp. from AFM)\n- Boost converter for larger gate drive on board\n- Add interface for external chip (tire sensors)\n- Add interface for non-packaged chip (pogo pins)\n- Add temperature, humidity, and pressure sensors\n- DONE: Solution Gate and Back Gate are switched on Socket!  Fix!\n- DONE: Need holes for magnets or something to preserve absolute positioning on AFM stage\n
 Wire Wire Line
 	20900 2600 21350 2600

Commit message: Renamed all of the processors in layout 2_15 so it is much easier to understand
Parts:
- renumbered U3 to CPU1, U7 to CPU2, U1 to MP1, U2 to MP2, U4 to MP3, U6 to MP4, U5 to SKT1
Changed lines of the file:
@@
 $EndDescr
 $Comp
-L Selection-Interface-rescue:68_PLCC_Socket_(8468-21B1-RK-TP) U5
+L Selection-Interface-rescue:68_PLCC_Socket_(8468-21B1-RK-TP) SKT1
 U 1 1 5913392C
 P 1900 4150
-F 0 "U5" H 1900 4050 50  0000 C CNN
+F 0 "SKT1" H 1900 4050 50  0000 C CNN
 F 1 "68_PLCC_Socket_(8468-21B1-RK-TP)" H 1900 4250 50  0000 C CNN
 F 2 "Custom_Footprint_Library:68_PLCC_Socket_(8468-21B1-RK-TP)" H 1900 4150 50  0001 C CNN
@@
 GND
 $Comp
-L Selection-Interface-rescue:CY8C42_(48_TQFP) U1
+L Selection-Interface-rescue:CY8C42_(48_TQFP) MP1
 U 1 1 599B549F
 P 23700 11550
-F 0 "U1" H 23700 11450 50  0000 C CNN
+F 0 "MP1" H 23700 11450 50  0000 C CNN
 F 1 "CY8C42_(48_TQFP)" H 23700 11650 50  0000 C CNN
 F 2 "Package_QFP:TQFP-48_7x7mm_P0.5mm" H 23700 11800 50  0001 C CNN
@@
 VDDD
 $Comp
-L Selection-Interface-rescue:CY8C58_(100_TQFP) U3
+L Selection-Interface-rescue:CY8C58_(100_TQFP) CPU1
 U 1 1 599B523D
 P 17500 2500
-F 0 "U3" H 17500 2400 50  0000 C CNN
+F 0 "CPU1" H 17500 2400 50  0000 C CNN
 F 1 "CY8C58_(100_TQFP)" H 17500 2600 50  0000 C CNN
 F 2 "Package_QFP:TQFP-100_14x14mm_P0.5mm" H 17500 3000 50  0001 C CNN
@@
 I9
 $Comp
-L Selection-Interface-rescue:CY8C42_(48_TQFP) U6
+L Selection-Interface-rescue:CY8C42_(48_TQFP) MP4
 U 1 1 599EBC26
 P 17100 11350
-F 0 "U6" H 17100 11250 50  0000 C CNN
+F 0 "MP4" H 17100 11250 50  0000 C CNN
 F 1 "CY8C42_(48_TQFP)" H 17100 11450 50  0000 C CNN
 F 2 "Package_QFP:TQFP-48_7x7mm_P0.5mm" H 17100 11600 50  0001 C CNN
@@
 S3
 $Comp
-L Selection-Interface-rescue:CY8C42_(48_TQFP) U2
+L Selection-Interface-rescue:CY8C42_(48_TQFP) MP2
 U 1 1 599EC71E
 P 23700 17250
-F 0 "U2" H 23700 17150 50  0000 C CNN
+F 0 "MP2" H 23700 17150 50  0000 C CNN
 F 1 "CY8C42_(48_TQFP)" H 23700 17350 50  0000 C CNN
 F 2 "Package_QFP:TQFP-48_7x7mm_P0.5mm" H 23700 17500 50  0001 C CNN
@@
 S1
 $Comp
-L Selection-Interface-rescue:CY8C42_(48_TQFP) U4
+L Selection-Interface-rescue:CY8C42_(48_TQFP) MP3
 U 1 1 599F47BA
 P 16850 17200
-F 0 "U4" H 16850 17100 50  0000 C CNN
+F 0 "MP3" H 16850 17100 50  0000 C CNN
 F 1 "CY8C42_(48_TQFP)" H 16850 17300 50  0000 C CNN
 F 2 "Package_QFP:TQFP-48_7x7mm_P0.5mm" H 16850 17450 50  0001 C CNN
@@
 VDDD
 $Comp
-L Selection-Interface-rescue:CY8C58_(100_TQFP) U7
+L Selection-Interface-rescue:CY8C58_(100_TQFP) CPU2
 U 1 1 599F6541
 P 26650 2650
-F 0 "U7" H 26650 2550 50  0000 C CNN
+F 0 "CPU2" H 26650 2550 50  0000 C CNN
 F 1 "CY8C58_(100_TQFP)" H 26650 2750 50  0000 C CNN
 F 2 "Package_QFP:TQFP-100_14x14mm_P0.5mm" H 26650 3150 50  0001 C CNN

Commit message: Renamed S1, S2, S3, S4 to SS2, SS1, DD2, DD1 respectively. This is because we have been using S4 and S2 as drain and source in the past. S1 and S3 have been unused but in theory could be used to select another device for simultaneous device measurements
Connections:
- net labels added: DD1, DD2, SS1, SS2
- net labels removed: S1, S2, S3, S4
- wire segments 289 -> 285
Changed lines of the file:
@@
 D32
 Text GLabel 25100 11200 2    39   Input ~ 0
-S2
+SS1
 Text GLabel 25100 11100 2    39   Input ~ 0
-S1
+SS2
 Text GLabel 17300 800  1    39   Input ~ 0
-S1
+SS2
 Text GLabel 17100 800  1    39   Input ~ 0
-S2
+SS1
 Text GLabel 15250 3500 0    39   Input ~ 0
 I1
@@
 I4
 Text GLabel 17000 4200 3    39   Input ~ 0
-I5
-Text GLabel 17900 4200 3    39   Input ~ 0
-I6
-Text GLabel 18100 4200 3    39   Input ~ 0
-I7
-Text GLabel 18300 4200 3    39   Input ~ 0
-I8
+SS2
 Text GLabel 18500 4200 3    39   Input ~ 0
 I9
@@
 D32
 Text GLabel 18500 11000 2    39   Input ~ 0
-S4
+DD1
 Text GLabel 18500 10900 2    39   Input ~ 0
-S3
+DD2
 $Comp
 L Selection-Interface-rescue:CY8C42_(48_TQFP) MP2
@@
 D64
 Text GLabel 25100 16900 2    39   Input ~ 0
-S2
+SS1
 Text GLabel 25100 16800 2    39   Input ~ 0
-S1
+SS2
 $Comp
 L Selection-Interface-rescue:CY8C42_(48_TQFP) MP3
@@
 D64
 Text GLabel 18250 16850 2    39   Input ~ 0
-S4
+DD1
 Text GLabel 18250 16750 2    39   Input ~ 0
-S3
+DD2
 Text GLabel 24400 1750 0    39   Input ~ 0
 I2C0_SCL
@@
 	26350 5000 26350 5300
 Text GLabel 26450 950  1    39   Input ~ 0
-S1
+SS2
 Text GLabel 26250 950  1    39   Input ~ 0
-S2
+SS1
 Text GLabel 24400 3650 0    39   Input ~ 0
 I1
@@
 I4
 Text GLabel 26150 4350 3    39   Input ~ 0
-I5
-Text GLabel 27050 4350 3    39   Input ~ 0
-I6
-Text GLabel 27250 4350 3    39   Input ~ 0
-I7
-Text GLabel 27450 4350 3    39   Input ~ 0
-I8
+SS2
 Text GLabel 27650 4350 3    39   Input ~ 0
 I9
@@
 	8650 2000 9150 2000
 Text GLabel 16900 800  1    39   Input ~ 0
-S3
+DD2
 Text GLabel 16700 800  1    39   Input ~ 0
-S4
+DD1
 Text GLabel 26050 950  1    39   Input ~ 0
-S3
+DD2
 Text GLabel 25850 950  1    39   Input ~ 0
-S4
+DD1
 Text GLabel 3900 1800 0    39   Input ~ 0
-S1
+SS2
 Text GLabel 3900 1900 0    39   Input ~ 0
-S2
+SS1
 Text GLabel 4400 1800 2    39   Input ~ 0
-S3
+DD2
 Text GLabel 4400 1900 2    39   Input ~ 0
-S4
+DD1
 Text GLabel 3900 1600 0    39   Input ~ 0
 LocalGates
@@
 Text GLabel 3050 3700 0    39   Input ~ 0
 I7
-Text GLabel 3050 3800 0    39   Input ~ 0
-I8
 Text GLabel 3050 3900 0    39   Input ~ 0
 I9
 Text GLabel 3150 3500 2    39   Input ~ 0
-S1
+SS2
 Text GLabel 3150 3100 2    39   Input ~ 0
 GND
@@
 BackGate
 Text GLabel 3150 3600 2    39   Input ~ 0
-S2
+SS1
 Text GLabel 3150 3700 2    39   Input ~ 0
-S3
-Text GLabel 3150 3800 2    39   Input ~ 0
-S4
+DD2
 Text GLabel 3050 4000 0    39   Input ~ 0
 I10
@@
 	3050 3400 3150 3400
 Wire Wire Line
-	3050 3500 3150 3500
-Wire Wire Line
-	3050 3600 3150 3600
-Wire Wire Line
-	3050 3700 3150 3700
-Wire Wire Line
-	3050 3800 3150 3800
-Wire Wire Line
 	4400 1400 4400 1500
 Connection ~ 4400 1600
@@
 BackGate
 Text GLabel 4800 5800 1    39   Input ~ 0
-S1
+SS2
 Text GLabel 5300 5800 1    39   Input ~ 0
-S2
+SS1
 Text GLabel 5800 5800 1    39   Input ~ 0
-S3
+DD2
 Text GLabel 6300 5800 1    39   Input ~ 0
-S4
+DD1
 Text GLabel 6800 5800 1    39   Input ~ 0
 I9
@@
 	1    0    0    -1
 $EndComp
+Text GLabel 3050 3800 0    39   Input ~ 0
+I8
+Text GLabel 3150 3800 2    39   Input ~ 0
+DD1
 $EndSCHEMATC

Commit message: Renamed I9, I10, I11, I12 to IO1, I02, IO3, IO4 respectively. This is because I will likely be moving some of them to different pins on CPU1/CPU2 because we discovered that I9 is currently not functional
Connections:
- net labels added: IO1, IO2, IO3, IO4
- net labels removed: I10, I11, I12, I9
Changed lines of the file:
@@
 SS2
 Text GLabel 18500 4200 3    39   Input ~ 0
-I9
+IO1
 $Comp
 L Selection-Interface-rescue:CY8C42_(48_TQFP) MP4
@@
 SS2
 Text GLabel 27650 4350 3    39   Input ~ 0
-I9
+IO1
 $Comp
 L Device:R R7
@@
 I7
 Text GLabel 3050 3900 0    39   Input ~ 0
-I9
+IO1
 Text GLabel 3150 3500 2    39   Input ~ 0
 SS2
@@
 DD2
 Text GLabel 3050 4000 0    39   Input ~ 0
-I10
+IO2
 Text GLabel 3050 4100 0    39   Input ~ 0
-I11
+IO3
 Text GLabel 3050 4200 0    39   Input ~ 0
-I12
+IO4
 Text GLabel 19800 3700 2    39   Input ~ 0
-I10
+IO2
 Text GLabel 19800 3200 2    39   Input ~ 0
-I11
+IO3
 Text GLabel 19800 1900 2    39   Input ~ 0
-I12
+IO4
 Text GLabel 28950 3850 2    39   Input ~ 0
-I10
+IO2
 Text GLabel 28950 3350 2    39   Input ~ 0
-I11
+IO3
 Text GLabel 28950 2050 2    39   Input ~ 0
-I12
+IO4
 Text GLabel 4350 2600 0    39   Input ~ 0
 BT1_RX
@@
 $EndComp
 Text GLabel 3900 2000 0    39   Input ~ 0
-I9
+IO1
 Text GLabel 3900 2100 0    39   Input ~ 0
-I10
+IO2
 Text GLabel 3900 2200 0    39   Input ~ 0
-I11
+IO3
 Text GLabel 3900 2300 0    39   Input ~ 0
-I12
+IO4
 Wire Wire Line
 	3050 3100 3150 3100
@@
 DD1
 Text GLabel 6800 5800 1    39   Input ~ 0
-I9
+IO1
 Text GLabel 7300 5800 1    39   Input ~ 0
-I10
+IO2
 Text GLabel 7800 5800 1    39   Input ~ 0
-I11
+IO3
 Text GLabel 8300 5800 1    39   Input ~ 0
-I12
+IO4
 $Comp
 L Selection-Interface-rescue:CONN_02X10 P6
