File: PCB Layouts/Layout 2_15/Selection Interface.sch (KiCad schematic (older format))
At the start: 132 parts, among them P1 CONN_01X02, P11 CONN_01X02, P12 CONN_01X02, P13 CONN_01X10, P14 CONN_01X02, P15 CONN_01X02, P16 CONN_01X02, P18 CONN_02X05, P19 CONN_02X05, P2 CONN_01X02, P21 CONN_02X05, P3 CONN_01X02, P4 CONN_01X02, P5 CONN_01X02, P6 CONN_02X10, P7 CONN_01X02, P8 CONN_02X04, P9 CONN_01X02, U8 USB_2.0_B, U9 USB_2.0_B

Commit message: Moved around IO1, IO2, and IO3 so that hopefully all of them will now be attached to functional pins on the cypress chips. Also moved some vias around to satisfy the default design rules checker. This board is in very good shape now and might be worth ordering.
Parts:
- renumbered U8 to USB1, U9 to USB2
Connections:
- wire segments 285 -> 282
Other:
- note added: "- Don’t have gates permanently connected to PSoCs\n- Break out I2C\n- Give Masters ability to reset Slaves\n- Add more optional TIA resistors\n- DONE: Give PSoCs more natural number labels\n- Communication between Masters\n- Clock sync between Masters\n- Resistor dividers for input measurements (esp. from AFM)\n- Boost converter for larger gate drive on board\n- Add interface for external chip (t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"
- note removed: "- Don’t have gates permanently connected to PSoCs\n- Break out I2C\n- Give Masters ability to reset Slaves\n- Add more optional TIA resistors\n- Give PSoCs more natural number labels\n- Communication between Masters\n- Clock sync between Masters\n- Resistor dividers for input measurements (esp. from AFM)\n- Boost converter for larger gate drive on board\n- Add interface for external chip (tire se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"
Changed lines of the file:
@@
 I1
 Text GLabel 15250 3700 0    39   Input ~ 0
-I2
+SolutionGate
 Text GLabel 16500 4200 3    39   Input ~ 0
-I3
+LocalGates
 Text GLabel 16800 4200 3    39   Input ~ 0
-I4
+BackGate
 Text GLabel 17000 4200 3    39   Input ~ 0
-SS2
-Text GLabel 18500 4200 3    39   Input ~ 0
 IO1
 $Comp
@@
 I1
 Text GLabel 24400 3850 0    39   Input ~ 0
-I2
+SolutionGate
 Text GLabel 25650 4350 3    39   Input ~ 0
-I3
+LocalGates
 Text GLabel 25950 4350 3    39   Input ~ 0
-I4
+BackGate
 Text GLabel 26150 4350 3    39   Input ~ 0
-SS2
-Text GLabel 27650 4350 3    39   Input ~ 0
 IO1
 $Comp
@@
 Text GLabel 3050 4200 0    39   Input ~ 0
 IO4
-Text GLabel 19800 3700 2    39   Input ~ 0
+Text GLabel 19800 3200 2    39   Input ~ 0
 IO2
-Text GLabel 19800 3200 2    39   Input ~ 0
-IO3
 Text GLabel 19800 1900 2    39   Input ~ 0
 IO4
-Text GLabel 28950 3850 2    39   Input ~ 0
+Text GLabel 28950 3350 2    39   Input ~ 0
 IO2
-Text GLabel 28950 3350 2    39   Input ~ 0
+Text GLabel 28950 1950 2    39   Input ~ 0
 IO3
 Text GLabel 28950 2050 2    39   Input ~ 0
@@
 Wire Wire Line
 	3050 3100 3150 3100
-Wire Wire Line
-	3050 3200 3150 3200
-Wire Wire Line
-	3050 3300 3150 3300
-Wire Wire Line
-	3050 3400 3150 3400
 Wire Wire Line
 	4400 1400 4400 1500
@@
 VDDD
 $Comp
-L Selection-Interface-rescue:USB_2.0_B U8
+L Selection-Interface-rescue:USB_2.0_B USB1
 U 1 1 59A082C2
 P 17300 5650
-F 0 "U8" H 17300 5700 60  0000 C CNN
+F 0 "USB1" H 17300 5700 60  0000 C CNN
 F 1 "USB_2.0_B" H 17300 5600 60  0000 C CNN
 F 2 "Custom_Footprint_Library:Micro_USB_2.0_B_SMD(10118192-0001LF)" H 17300 5650 60  0001 C CNN
@@
 	17250 5150 17300 5150
 $Comp
-L Selection-Interface-rescue:USB_2.0_B U9
+L Selection-Interface-rescue:USB_2.0_B USB2
 U 1 1 59A0C386
 P 26450 5850
-F 0 "U9" H 26450 5900 60  0000 C CNN
+F 0 "USB2" H 26450 5900 60  0000 C CNN
 F 1 "USB_2.0_B" H 26450 5800 60  0000 C CNN
 F 2 "Custom_Footprint_Library:Micro_USB_2.0_B_SMD(10118192-0001LF)" H 26450 5850 60  0001 C CNN
@@
 	5600 3700 5150 3700
 Text Notes 6600 3750 0    60   ~ 0
-- Don’t have gates permanently connected to PSoCs\n- Break out I2C\n- Give Masters ability to reset Slaves\n- Add more optional TIA resistors\n- Give PSoCs more natural number labels\n- Communication between Masters\n- Clock sync between Masters\n- Resistor dividers for input measurements (esp. from AFM)\n- Boost converter for larger gate drive on board\n- Add interface for external chip (tire sensors)\n- Add interface for non-packaged chip (pogo pins)\n- Add temperature, humidity, and pressure sensors\n- DONE: Solution Gate and Back Gate are switched on Socket!  Fix!\n- DONE: Need holes for magnets or something to preserve absolute positioning on AFM stage\n
+- Don’t have gates permanently connected to PSoCs\n- Break out I2C\n- Give Masters ability to reset Slaves\n- Add more optional TIA resistors\n- DONE: Give PSoCs more natural number labels\n- Communication between Masters\n- Clock sync between Masters\n- Resistor dividers for input measurements (esp. from AFM)\n- Boost converter for larger gate drive on board\n- Add interface for external chip (tire sensors)\n- Add interface for non-packaged chip (pogo pins)\n- Add temperature, humidity, and pressure sensors\n- DONE: Solution Gate and Back Gate are switched on Socket!  Fix!\n- DONE: Need holes for magnets or something to preserve absolute positioning on AFM stage\n
 Wire Wire Line
 	20900 2600 21350 2600
@@
 Text GLabel 3150 3800 2    39   Input ~ 0
 DD1
+Text GLabel 19800 1800 2    39   Input ~ 0
+IO3
 $EndSCHEMATC
