File: PCB Layouts/Layout 2_15/Selection Interface.sch (KiCad schematic (older format))
At the start: 132 parts, among them P1 CONN_01X02, P11 CONN_01X02, P12 CONN_01X02, P13 CONN_01X10, P14 CONN_01X02, P15 CONN_01X02, P16 CONN_01X02, P18 CONN_02X05, P19 CONN_02X05, P2 CONN_01X02, P21 CONN_02X05, P3 CONN_01X02, P4 CONN_01X02, P5 CONN_01X02, P6 CONN_02X10, P7 CONN_01X02, P8 CONN_02X04, P9 CONN_01X02

Commit message: Renamed the multiplexers in Layout 2_15
Parts:
- renumbered MP4 to MP2, MP2 to MP3, MP3 to MP4
Changed lines of the file:
@@
 IO1
 $Comp
-L Selection-Interface-rescue:CY8C42_(48_TQFP) MP4
+L Selection-Interface-rescue:CY8C42_(48_TQFP) MP2
 U 1 1 599EBC26
 P 17100 11350
-F 0 "MP4" H 17100 11250 50  0000 C CNN
+F 0 "MP2" H 17100 11250 50  0000 C CNN
 F 1 "CY8C42_(48_TQFP)" H 17100 11450 50  0000 C CNN
 F 2 "Package_QFP:TQFP-48_7x7mm_P0.5mm" H 17100 11600 50  0001 C CNN
@@
 DD2
 $Comp
-L Selection-Interface-rescue:CY8C42_(48_TQFP) MP2
+L Selection-Interface-rescue:CY8C42_(48_TQFP) MP3
 U 1 1 599EC71E
 P 23700 17250
-F 0 "MP2" H 23700 17150 50  0000 C CNN
+F 0 "MP3" H 23700 17150 50  0000 C CNN
 F 1 "CY8C42_(48_TQFP)" H 23700 17350 50  0000 C CNN
 F 2 "Package_QFP:TQFP-48_7x7mm_P0.5mm" H 23700 17500 50  0001 C CNN
@@
 SS2
 $Comp
-L Selection-Interface-rescue:CY8C42_(48_TQFP) MP3
+L Selection-Interface-rescue:CY8C42_(48_TQFP) MP4
 U 1 1 599F47BA
 P 16850 17200
-F 0 "MP3" H 16850 17100 50  0000 C CNN
+F 0 "MP4" H 16850 17100 50  0000 C CNN
 F 1 "CY8C42_(48_TQFP)" H 16850 17300 50  0000 C CNN
 F 2 "Package_QFP:TQFP-48_7x7mm_P0.5mm" H 16850 17450 50  0001 C CNN

Commit message: Added a new compoent to try to reduce the area taken up by programming headers. Began making some wiring changes to facilitate this
Parts:
- added PROG2: Conn_02x06_Odd_Even, Connector_PinHeader_2.54mm:PinHeader_2x06_P2.54mm_Vertical_SMD, symbol Connector_Generic:Conn_02x06_Odd_Even
- renumbered SKT1 to SOCKET1
Changed lines of the file:
@@
 $EndDescr
 $Comp
-L Selection-Interface-rescue:68_PLCC_Socket_(8468-21B1-RK-TP) SKT1
+L Selection-Interface-rescue:68_PLCC_Socket_(8468-21B1-RK-TP) SOCKET1
 U 1 1 5913392C
 P 1900 4150
-F 0 "SKT1" H 1900 4050 50  0000 C CNN
+F 0 "SOCKET1" H 1900 4050 50  0000 C CNN
 F 1 "68_PLCC_Socket_(8468-21B1-RK-TP)" H 1900 4250 50  0000 C CNN
 F 2 "Custom_Footprint_Library:68_PLCC_Socket_(8468-21B1-RK-TP)" H 1900 4150 50  0001 C CNN
@@
 Text GLabel 15700 11600 0    39   Input ~ 0
 D16
-Text GLabel 16650 12800 3    39   Input ~ 0
+Text GLabel 16650 13050 3    39   Input ~ 0
 D17P
-Text GLabel 16850 12950 3    39   Input ~ 0
+Text GLabel 16850 13050 3    39   Input ~ 0
 D18P
 Text GLabel 16950 12400 3    39   Input ~ 0
@@
 Text GLabel 15450 17450 0    39   Input ~ 0
 D48
-Text GLabel 16400 18650 3    39   Input ~ 0
-D49P
-Text GLabel 16600 18800 3    39   Input ~ 0
+Text GLabel 16600 18900 3    39   Input ~ 0
 D50P
 Text GLabel 16700 18250 3    39   Input ~ 0
@@
 	22700 13150 23450 13150
 Text GLabel 20550 16750 2    39   Input ~ 0
-SWDCLK4
+SWDCLK3
 Text GLabel 20550 16650 2    39   Input ~ 0
-SWDIO4
+SWDIO3
 Text GLabel 20550 16850 2    39   Input ~ 0
-XRES4
+XRES3
 Text GLabel 18500 10800 2    39   Input ~ 0
 XRES2
@@
 	14950 18650 16400 18650
 Text GLabel 14950 18650 0    39   Input ~ 0
-SWDIO3
+SWDIO4
 Text GLabel 14850 18800 0    39   Input ~ 0
-SWDCLK3
+SWDCLK4
 Text GLabel 18250 16650 2    39   Input ~ 0
-XRES3
-Text GLabel 25100 16700 2    39   Input ~ 0
 XRES4
+Text GLabel 25100 16700 2    39   Input ~ 0
+XRES3
 Text GLabel 21800 18700 0    39   Input ~ 0
-SWDIO4
+SWDIO3
 Text GLabel 21700 18850 0    39   Input ~ 0
-SWDCLK4
+SWDCLK3
 Text GLabel 23600 3350 0    39   Input ~ 0
 SWDIO6
@@
 $EndComp
 Text GLabel 20050 16650 0    39   Input ~ 0
-SWDIO3
+SWDIO4
 Text GLabel 20050 16750 0    39   Input ~ 0
-SWDCLK3
+SWDCLK4
 Text GLabel 20050 16850 0    39   Input ~ 0
-XRES3
+XRES4
 Text GLabel 20050 16950 0    39   Input ~ 0
 VSSD
@@
 Text GLabel 19800 1800 2    39   Input ~ 0
 IO3
+$Comp
+L Connector_Generic:Conn_02x06_Odd_Even PROG2
+U 1 1 5DA1458B
+P 4050 4600
+F 0 "PROG2" H 4100 5017 50  0000 C CNN
+F 1 "Conn_02x06_Odd_Even" H 4100 4926 50  0000 C CNN
+F 2 "Connector_PinHeader_2.54mm:PinHeader_2x06_P2.54mm_Vertical_SMD" H 4050 4600 50  0001 C CNN
+F 3 "~" H 4050 4600 50  0001 C CNN
+	1    4050 4600
+	1    0    0    -1
+$EndComp
+Text GLabel 3850 4400 0    50   Input ~ 0
+SWDCLK1
+Text GLabel 3850 4500 0    50   Input ~ 0
+SWDCLK2
+Text GLabel 3850 4600 0    50   Input ~ 0
+SWDCLK3
+Text GLabel 3850 4700 0    50   Input ~ 0
+SWDCLK4
+Text GLabel 3850 4800 0    50   Input ~ 0
+SWDCLK5
+Text GLabel 3850 4900 0    50   Input ~ 0
+SWDCLK6
+Text GLabel 4350 4400 2    50   Input ~ 0
+SWDIO1
+Text GLabel 4350 4500 2    50   Input ~ 0
+SWDIO2
+Text GLabel 4350 4600 2    50   Input ~ 0
+SWDIO3
+Text GLabel 4350 4700 2    50   Input ~ 0
+SWDIO4
+Text GLabel 4350 4800 2    50   Input ~ 0
+SWDIO5
+Text GLabel 4350 4900 2    50   Input ~ 0
+SWDIO6
+Text GLabel 16400 18900 3    39   Input ~ 0
+D49P
 $EndSCHEMATC

Commit message: Did more routing on layout 2_15
Parts:
- removed P19, P21: CONN_02X05, Connector_PinHeader_2.54mm:PinHeader_2x05_P2.54mm_Vertical_SMD, symbol Selection-Interface-rescue:CONN_02X05
- added MH4: MountingHole, Custom_Footprint_Library:MountingHole_5.1mm, symbol Mechanical:MountingHole
Connections:
- net labels added: SWDCLK, SWDIO, XRES
- net labels removed: XRES1, XRES2, XRES3, XRES4, XRES5, XRES6
Changed lines of the file:
@@
 	1    0    0    -1
 $EndComp
-Text GLabel 20550 16950 2    39   Input ~ 0
-VSSD
-Text GLabel 20550 17050 2    39   Input ~ 0
-VDDD
 Text GLabel 15250 1600 0    39   Input ~ 0
 I2C0_SCL
@@
 $EndComp
 Text GLabel 25100 11000 2    39   Input ~ 0
-XRES1
+XRES
 Text GLabel 22900 13000 0    39   Input ~ 0
 SWDIO1
@@
 Wire Wire Line
 	22700 13150 23450 13150
-Text GLabel 20550 16750 2    39   Input ~ 0
-SWDCLK3
-Text GLabel 20550 16650 2    39   Input ~ 0
-SWDIO3
-Text GLabel 20550 16850 2    39   Input ~ 0
-XRES3
 Text GLabel 18500 10800 2    39   Input ~ 0
-XRES2
+XRES
 Text GLabel 15200 12800 0    39   Input ~ 0
 SWDIO2
@@
 SWDCLK4
 Text GLabel 18250 16650 2    39   Input ~ 0
-XRES4
+XRES
 Text GLabel 25100 16700 2    39   Input ~ 0
-XRES3
+XRES
 Text GLabel 21800 18700 0    39   Input ~ 0
 SWDIO3
@@
 SWDCLK6
 Text GLabel 23600 3550 0    39   Input ~ 0
-XRES6
+XRES
 Text GLabel 14450 3200 0    39   Input ~ 0
 SWDIO5
@@
 SWDCLK5
 Text GLabel 14450 3400 0    39   Input ~ 0
-XRES5
-$Comp
-L Selection-Interface-rescue:CONN_02X05 P21
-U 1 1 59A42FA7
-P 20300 16850
-F 0 "P21" H 20300 17150 50  0000 C CNN
-F 1 "CONN_02X05" H 20300 16550 50  0000 C CNN
-F 2 "Connector_PinHeader_2.54mm:PinHeader_2x05_P2.54mm_Vertical_SMD" H 20300 15650 50  0001 C CNN
-F 3 "" H 20300 15650 50  0000 C CNN
-	1    20300 16850
-	1    0    0    -1
-$EndComp
-Text GLabel 20050 16650 0    39   Input ~ 0
-SWDIO4
-Text GLabel 20050 16750 0    39   Input ~ 0
-SWDCLK4
-Text GLabel 20050 16850 0    39   Input ~ 0
-XRES4
-Text GLabel 20050 16950 0    39   Input ~ 0
-VSSD
-Text GLabel 20050 17050 0    39   Input ~ 0
-VDDD
-Text GLabel 20700 11150 2    39   Input ~ 0
-VSSD
-Text GLabel 20700 11250 2    39   Input ~ 0
-VDDD
-Text GLabel 20700 10950 2    39   Input ~ 0
-SWDCLK1
-Text GLabel 20700 10850 2    39   Input ~ 0
-SWDIO1
-Text GLabel 20700 11050 2    39   Input ~ 0
-XRES1
-$Comp
-L Selection-Interface-rescue:CONN_02X05 P19
-U 1 1 59A43DA9
-P 20450 11050
-F 0 "P19" H 20450 11350 50  0000 C CNN
-F 1 "CONN_02X05" H 20450 10750 50  0000 C CNN
-F 2 "Connector_PinHeader_2.54mm:PinHeader_2x05_P2.54mm_Vertical_SMD" H 20450 9850 50  0001 C CNN
-F 3 "" H 20450 9850 50  0000 C CNN
-	1    20450 11050
-	1    0    0    -1
-$EndComp
-Text GLabel 20200 10850 0    39   Input ~ 0
-SWDIO2
-Text GLabel 20200 10950 0    39   Input ~ 0
-SWDCLK2
-Text GLabel 20200 11050 0    39   Input ~ 0
-XRES2
-Text GLabel 20200 11150 0    39   Input ~ 0
-VSSD
-Text GLabel 20200 11250 0    39   Input ~ 0
-VDDD
+XRES
 Text GLabel 22350 4600 2    39   Input ~ 0
 VSSD
@@
 VDDD
 Text GLabel 22350 4400 2    39   Input ~ 0
-SWDCLK6
+SWDCLK
 Text GLabel 22350 4300 2    39   Input ~ 0
-SWDIO6
+SWDIO
 Text GLabel 22350 4500 2    39   Input ~ 0
-XRES6
+XRES
 $Comp
 L Selection-Interface-rescue:CONN_02X05 P18
@@
 $EndComp
 Text GLabel 21850 4300 0    39   Input ~ 0
-SWDIO5
+SWDIO
 Text GLabel 21850 4400 0    39   Input ~ 0
-SWDCLK5
+SWDCLK
 Text GLabel 21850 4500 0    39   Input ~ 0
-XRES5
+XRES
 Text GLabel 21850 4600 0    39   Input ~ 0
 VSSD
@@
 Text GLabel 16400 18900 3    39   Input ~ 0
 D49P
+$Comp
+L Mechanical:MountingHole MH4
+U 1 1 5DA3CFD1
+P 10100 5500
+F 0 "MH4" H 10200 5546 50  0000 L CNN
+F 1 "MountingHole" H 10200 5455 50  0000 L CNN
+F 2 "Custom_Footprint_Library:MountingHole_5.1mm" H 10100 5500 50  0001 C CNN
+F 3 "~" H 10100 5500 50  0001 C CNN
+	1    10100 5500
+	1    0    0    -1
+$EndComp
 $EndSCHEMATC

Commit message: Added new schematic symbol for a new multiplexer processor that has more GPIO pins. Started modifying signal routing for the slightly different pinout
Parts:
- removed MP1: CY8C42_(48_TQFP), Package_QFP:TQFP-48_7x7mm_P0.5mm, symbol Selection-Interface-rescue:CY8C42_(48_TQFP)
- added MP1: CY8C4245AZI-M433(48_TQPF), Package_QFP:TQFP-48_7x7mm_P0.5mm, symbol Custom_Schematic_Library:CY8C4245AZI-M433(48_TQPF)
Connections:
- net labels removed: D17P, D18P
Changed lines of the file:
@@
 Text GLabel 1150 1100 0    39   Input ~ 0
 GND
-$Comp
-L Selection-Interface-rescue:CY8C42_(48_TQFP) MP1
-U 1 1 599B549F
-P 23700 11550
-F 0 "MP1" H 23700 11450 50  0000 C CNN
-F 1 "CY8C42_(48_TQFP)" H 23700 11650 50  0000 C CNN
-F 2 "Package_QFP:TQFP-48_7x7mm_P0.5mm" H 23700 11800 50  0001 C CNN
-F 3 "DOCUMENTATION" H 23700 11300 50  0001 C CNN
-	1    23700 11550
-	1    0    0    -1
-$EndComp
 Text GLabel 15250 1600 0    39   Input ~ 0
 I2C0_SCL
@@
 VDDIO
 Text GLabel 23950 12600 3    39   Input ~ 0
-VDDD
-Text GLabel 23350 12600 3    39   Input ~ 0
+VDDIO
+Text GLabel 22300 11900 0    39   Input ~ 0
 VSSD
 Text GLabel 24150 10500 1    39   Input ~ 0
@@
 Text GLabel 22300 11800 0    39   Input ~ 0
 D16
-Text GLabel 23250 13000 3    39   Input ~ 0
+Text GLabel 23550 12600 3    39   Input ~ 0
 D17
-Text GLabel 23450 13150 3    39   Input ~ 0
+Text GLabel 23650 12600 3    39   Input ~ 0
 D18
-Text GLabel 23550 12600 3    39   Input ~ 0
+Text GLabel 23750 12600 3    39   Input ~ 0
 D19
-Text GLabel 23650 12600 3    39   Input ~ 0
+Text GLabel 23850 12600 3    39   Input ~ 0
 D20
-Text GLabel 23750 12600 3    39   Input ~ 0
+Text GLabel 24050 12600 3    39   Input ~ 0
 D21
-Text GLabel 23850 12600 3    39   Input ~ 0
+Text GLabel 24150 12600 3    39   Input ~ 0
 D22
-Text GLabel 24050 12600 3    39   Input ~ 0
+Text GLabel 24250 12600 3    39   Input ~ 0
 D23
-Text GLabel 24150 12600 3    39   Input ~ 0
+Text GLabel 25100 12100 2    39   Input ~ 0
 D24
-Text GLabel 24250 12600 3    39   Input ~ 0
+Text GLabel 25100 12000 2    39   Input ~ 0
 D25
-Text GLabel 25100 12100 2    39   Input ~ 0
+Text GLabel 25100 11900 2    39   Input ~ 0
 D26
 Text GLabel 25100 11400 2    39   Input ~ 0
@@
 D16
 Text GLabel 16650 13050 3    39   Input ~ 0
-D17P
+D17
 Text GLabel 16850 13050 3    39   Input ~ 0
-D18P
+D18
 Text GLabel 16950 12400 3    39   Input ~ 0
 D19
@@
 	1    0    0    -1
 $EndComp
+$Comp
+L Custom_Schematic_Library:CY8C4245AZI-M433(48_TQPF) MP1
+U 1 1 5DBAE2AD
+P 23700 11550
+F 0 "MP1" H 23700 11450 50  0000 C CNN
+F 1 "CY8C4245AZI-M433(48_TQPF)" H 23700 11650 50  0000 C CNN
+F 2 "Package_QFP:TQFP-48_7x7mm_P0.5mm" H 23700 11550 50  0001 C CNN
+F 3 "" H 23700 11550 50  0001 C CNN
+	1    23700 11550
+	1    0    0    -1
+$EndComp

Commit message: Updated Red PCB layout so all MUXes fit the new pinout
Parts:
- removed MP2, MP3, MP4: CY8C42_(48_TQFP), Package_QFP:TQFP-48_7x7mm_P0.5mm, symbol Selection-Interface-rescue:CY8C42_(48_TQFP)
- added MP2, MP3, MP4: CY8C4245AZI-M433(48_TQPF), Package_QFP:TQFP-48_7x7mm_P0.5mm, symbol Custom_Schematic_Library:CY8C4245AZI-M433(48_TQPF)
Connections:
- net labels removed: D49P, D50P
Changed lines of the file:
@@
 SS1
 Text GLabel 25100 11100 2    39   Input ~ 0
-SS2
+DD1
 Text GLabel 17300 800  1    39   Input ~ 0
-SS2
+DD1
 Text GLabel 17100 800  1    39   Input ~ 0
 SS1
@@
 Text GLabel 17000 4200 3    39   Input ~ 0
 IO1
-$Comp
-L Selection-Interface-rescue:CY8C42_(48_TQFP) MP2
-U 1 1 599EBC26
-P 17100 11350
-F 0 "MP2" H 17100 11250 50  0000 C CNN
-F 1 "CY8C42_(48_TQFP)" H 17100 11450 50  0000 C CNN
-F 2 "Package_QFP:TQFP-48_7x7mm_P0.5mm" H 17100 11600 50  0001 C CNN
-F 3 "DOCUMENTATION" H 17100 11100 50  0001 C CNN
-	1    17100 11350
-	1    0    0    -1
-$EndComp
 Text GLabel 15700 11900 0    39   Input ~ 0
 I2C0_SCL
@@
 I2C0_SDA
 Text GLabel 17350 12400 3    39   Input ~ 0
-VDDD
-Text GLabel 16750 12400 3    39   Input ~ 0
+VDDIO
+Text GLabel 15700 11700 0    39   Input ~ 0
 VSSD
 Text GLabel 17550 10300 1    39   Input ~ 0
@@
 Text GLabel 15700 11600 0    39   Input ~ 0
 D16
-Text GLabel 16650 13050 3    39   Input ~ 0
+Text GLabel 16950 12400 3    39   Input ~ 0
 D17
-Text GLabel 16850 13050 3    39   Input ~ 0
+Text GLabel 17050 12400 3    39   Input ~ 0
 D18
-Text GLabel 16950 12400 3    39   Input ~ 0
+Text GLabel 17150 12400 3    39   Input ~ 0
 D19
-Text GLabel 17050 12400 3    39   Input ~ 0
+Text GLabel 17250 12400 3    39   Input ~ 0
 D20
-Text GLabel 17150 12400 3    39   Input ~ 0
+Text GLabel 17450 12400 3    39   Input ~ 0
 D21
-Text GLabel 17250 12400 3    39   Input ~ 0
+Text GLabel 17550 12400 3    39   Input ~ 0
 D22
-Text GLabel 17450 12400 3    39   Input ~ 0
+Text GLabel 17650 12400 3    39   Input ~ 0
 D23
-Text GLabel 17550 12400 3    39   Input ~ 0
+Text GLabel 18500 11900 2    39   Input ~ 0
 D24
-Text GLabel 17650 12400 3    39   Input ~ 0
+Text GLabel 18500 11800 2    39   Input ~ 0
 D25
-Text GLabel 18500 11900 2    39   Input ~ 0
+Text GLabel 18500 11700 2    39   Input ~ 0
 D26
 Text GLabel 18500 11200 2    39   Input ~ 0
@@
 D32
 Text GLabel 18500 11000 2    39   Input ~ 0
-DD1
+SS2
 Text GLabel 18500 10900 2    39   Input ~ 0
 DD2
-$Comp
-L Selection-Interface-rescue:CY8C42_(48_TQFP) MP3
-U 1 1 599EC71E
-P 23700 17250
-F 0 "MP3" H 23700 17150 50  0000 C CNN
-F 1 "CY8C42_(48_TQFP)" H 23700 17350 50  0000 C CNN
-F 2 "Package_QFP:TQFP-48_7x7mm_P0.5mm" H 23700 17500 50  0001 C CNN
-F 3 "DOCUMENTATION" H 23700 17000 50  0001 C CNN
-	1    23700 17250
-	1    0    0    -1
-$EndComp
 Text GLabel 22300 17800 0    39   Input ~ 0
 I2C0_SCL
@@
 I2C0_SDA
 Text GLabel 23950 18300 3    39   Input ~ 0
-VDDD
-Text GLabel 23350 18300 3    39   Input ~ 0
+VDDIO
+Text GLabel 22300 17600 0    39   Input ~ 0
 VSSD
 Text GLabel 24150 16200 1    39   Input ~ 0
@@
 Text GLabel 22300 17500 0    39   Input ~ 0
 D48
-Text GLabel 23250 18700 3    39   Input ~ 0
+Text GLabel 23550 18300 3    39   Input ~ 0
 D49
-Text GLabel 23450 18850 3    39   Input ~ 0
+Text GLabel 23650 18300 3    39   Input ~ 0
 D50
-Text GLabel 23550 18300 3    39   Input ~ 0
+Text GLabel 23750 18300 3    39   Input ~ 0
 D51
-Text GLabel 23650 18300 3    39   Input ~ 0
+Text GLabel 23850 18300 3    39   Input ~ 0
 D52
-Text GLabel 23750 18300 3    39   Input ~ 0
+Text GLabel 24050 18300 3    39   Input ~ 0
 D53
-Text GLabel 23850 18300 3    39   Input ~ 0
+Text GLabel 24150 18300 3    39   Input ~ 0
 D54
-Text GLabel 24050 18300 3    39   Input ~ 0
+Text GLabel 24250 18300 3    39   Input ~ 0
 D55
-Text GLabel 24150 18300 3    39   Input ~ 0
+Text GLabel 25100 17800 2    39   Input ~ 0
 D56
-Text GLabel 24250 18300 3    39   Input ~ 0
+Text GLabel 25100 17700 2    39   Input ~ 0
 D57
-Text GLabel 25100 17800 2    39   Input ~ 0
+Text GLabel 25100 17600 2    39   Input ~ 0
 D58
 Text GLabel 25100 17100 2    39   Input ~ 0
@@
 SS1
 Text GLabel 25100 16800 2    39   Input ~ 0
-SS2
-$Comp
-L Selection-Interface-rescue:CY8C42_(48_TQFP) MP4
-U 1 1 599F47BA
-P 16850 17200
-F 0 "MP4" H 16850 17100 50  0000 C CNN
-F 1 "CY8C42_(48_TQFP)" H 16850 17300 50  0000 C CNN
-F 2 "Package_QFP:TQFP-48_7x7mm_P0.5mm" H 16850 17450 50  0001 C CNN
-F 3 "DOCUMENTATION" H 16850 16950 50  0001 C CNN
-	1    16850 17200
-	1    0    0    -1
-$EndComp
+DD1
 Text GLabel 15450 17750 0    39   Input ~ 0
 I2C0_SCL
@@
 I2C0_SDA
 Text GLabel 17100 18250 3    39   Input ~ 0
-VDDD
-Text GLabel 16500 18250 3    39   Input ~ 0
+VDDIO
+Text GLabel 15450 17550 0    39   Input ~ 0
 VSSD
 Text GLabel 17300 16150 1    39   Input ~ 0
@@
 Text GLabel 15450 17450 0    39   Input ~ 0
 D48
-Text GLabel 16600 18900 3    39   Input ~ 0
-D50P
-Text GLabel 16700 18250 3    39   Input ~ 0
+Text GLabel 16800 18250 3    39   Input ~ 0
+D50
+Text GLabel 16900 18250 3    39   Input ~ 0
 D51
-Text GLabel 16800 18250 3    39   Input ~ 0
+Text GLabel 17000 18250 3    39   Input ~ 0
 D52
-Text GLabel 16900 18250 3    39   Input ~ 0
+Text GLabel 17200 18250 3    39   Input ~ 0
 D53
-Text GLabel 17000 18250 3    39   Input ~ 0
+Text GLabel 17300 18250 3    39   Input ~ 0
 D54
-Text GLabel 17200 18250 3    39   Input ~ 0
+Text GLabel 17400 18250 3    39   Input ~ 0
 D55
-Text GLabel 17300 18250 3    39   Input ~ 0
+Text GLabel 18250 17750 2    39   Input ~ 0
 D56
-Text GLabel 17400 18250 3    39   Input ~ 0
+Text GLabel 18250 17650 2    39   Input ~ 0
 D57
-Text GLabel 18250 17750 2    39   Input ~ 0
+Text GLabel 18250 17550 2    39   Input ~ 0
 D58
 Text GLabel 18250 17050 2    39   Input ~ 0
@@
 D64
 Text GLabel 18250 16850 2    39   Input ~ 0
-DD1
+SS2
 Text GLabel 18250 16750 2    39   Input ~ 0
 DD2
@@
 	26350 5000 26350 5300
 Text GLabel 26450 950  1    39   Input ~ 0
-SS2
+DD1
 Text GLabel 26250 950  1    39   Input ~ 0
 SS1
@@
 DD2
 Text GLabel 16700 800  1    39   Input ~ 0
-DD1
+SS2
 Text GLabel 26050 950  1    39   Input ~ 0
 DD2
 Text GLabel 25850 950  1    39   Input ~ 0
+SS2
+Text GLabel 3900 1800 0    39   Input ~ 0
 DD1
-Text GLabel 3900 1800 0    39   Input ~ 0
-SS2
 Text GLabel 3900 1900 0    39   Input ~ 0
 SS1
@@
 DD2
 Text GLabel 4400 1900 2    39   Input ~ 0
-DD1
+SS2
 Text GLabel 3900 1600 0    39   Input ~ 0
 LocalGates
@@
 BackGate
 Text GLabel 4800 5800 1    39   Input ~ 0
-SS2
+DD1
 Text GLabel 5300 5800 1    39   Input ~ 0
 SS1
@@
 DD2
 Text GLabel 6300 5800 1    39   Input ~ 0
-DD1
+SS2
 Text GLabel 6800 5800 1    39   Input ~ 0
 IO1
@@
 Text GLabel 4350 4900 2    50   Input ~ 0
 SWDIO6
-Text GLabel 16400 18900 3    39   Input ~ 0
-D49P
+Text GLabel 16700 18250 3    39   Input ~ 0
+D49
 $Comp
 L Mechanical:MountingHole MH4
@@
 	1    0    0    -1
 $EndComp
+$Comp
+L Custom_Schematic_Library:CY8C4245AZI-M433(48_TQPF) MP2
+U 1 1 5DAF5D07
+P 17100 11350
+F 0 "MP2" H 17100 11250 50  0000 C CNN
+F 1 "CY8C4245AZI-M433(48_TQPF)" H 17100 11500 50  0000 C CNN
+F 2 "Package_QFP:TQFP-48_7x7mm_P0.5mm" H 17100 11350 50  0001 C CNN
+F 3 "" H 17100 11350 50  0001 C CNN
+	1    17100 11350
+	1    0    0    -1
+$EndComp
+$Comp
+L Custom_Schematic_Library:CY8C4245AZI-M433(48_TQPF) MP3
+U 1 1 5DB30235
+P 23700 17250
+F 0 "MP3" H 23700 17150 50  0000 C CNN
+F 1 "CY8C4245AZI-M433(48_TQPF)" H 23700 17350 50  0000 C CNN
+F 2 "Package_QFP:TQFP-48_7x7mm_P0.5mm" H 23700 17250 50  0001 C CNN
+F 3 "" H 23700 17250 50  0001 C CNN
+	1    23700 17250
+	1    0    0    -1
+$EndComp
+$Comp
+L Custom_Schematic_Library:CY8C4245AZI-M433(48_TQPF) MP4
+U 1 1 5DB85BD2
+P 16850 17200
+F 0 "MP4" H 16850 17100 50  0000 C CNN
+F 1 "CY8C4245AZI-M433(48_TQPF)" H 16850 17300 50  0000 C CNN
+F 2 "Package_QFP:TQFP-48_7x7mm_P0.5mm" H 16850 17200 50  0001 C CNN
+F 3 "" H 16850 17200 50  0001 C CNN
+	1    16850 17200
+	1    0    0    -1
+$EndComp

Commit message: Reverted a signal-name change made on the layout. I realized it is impossible for a signle MUX to route the signals for SS1 and DD1. The source and drain would be shorted out if I tried to do that
Changed lines of the file:
@@
 SS1
 Text GLabel 25100 11100 2    39   Input ~ 0
-DD1
+SS2
 Text GLabel 17300 800  1    39   Input ~ 0
-DD1
+SS2
 Text GLabel 17100 800  1    39   Input ~ 0
 SS1
@@
 D32
 Text GLabel 18500 11000 2    39   Input ~ 0
-SS2
+DD1
 Text GLabel 18500 10900 2    39   Input ~ 0
 DD2
@@
 SS1
 Text GLabel 25100 16800 2    39   Input ~ 0
-DD1
+SS2
 Text GLabel 15450 17750 0    39   Input ~ 0
 I2C0_SCL
@@
 D64
 Text GLabel 18250 16850 2    39   Input ~ 0
-SS2
+DD1
 Text GLabel 18250 16750 2    39   Input ~ 0
 DD2
@@
 	26350 5000 26350 5300
 Text GLabel 26450 950  1    39   Input ~ 0
-DD1
+SS2
 Text GLabel 26250 950  1    39   Input ~ 0
 SS1
@@
 DD2
 Text GLabel 16700 800  1    39   Input ~ 0
-SS2
+DD1
 Text GLabel 26050 950  1    39   Input ~ 0
 DD2
 Text GLabel 25850 950  1    39   Input ~ 0
+DD1
+Text GLabel 3900 1800 0    39   Input ~ 0
 SS2
-Text GLabel 3900 1800 0    39   Input ~ 0
-DD1
 Text GLabel 3900 1900 0    39   Input ~ 0
 SS1
@@
 DD2
 Text GLabel 4400 1900 2    39   Input ~ 0
-SS2
+DD1
 Text GLabel 3900 1600 0    39   Input ~ 0
 LocalGates
@@
 BackGate
 Text GLabel 4800 5800 1    39   Input ~ 0
-DD1
+SS2
 Text GLabel 5300 5800 1    39   Input ~ 0
 SS1
@@
 DD2
 Text GLabel 6300 5800 1    39   Input ~ 0
-SS2
+DD1
 Text GLabel 6800 5800 1    39   Input ~ 0
 IO1

Commit message: Renamed device selectors to MUX1, MUX2, MUX3, MUX4
Parts:
- renumbered MP1 to MUX1, MP2 to MUX2, MP3 to MUX3, MP4 to MUX4
Changed lines of the file:
@@
 $EndComp
 $Comp
-L Custom_Schematic_Library:CY8C4245AZI-M433(48_TQPF) MP1
+L Custom_Schematic_Library:CY8C4245AZI-M433(48_TQPF) MUX1
 U 1 1 5DBAE2AD
 P 23700 11550
-F 0 "MP1" H 23700 11450 50  0000 C CNN
+F 0 "MUX1" H 23700 11450 50  0000 C CNN
 F 1 "CY8C4245AZI-M433(48_TQPF)" H 23700 11650 50  0000 C CNN
 F 2 "Package_QFP:TQFP-48_7x7mm_P0.5mm" H 23700 11550 50  0001 C CNN
@@
 $EndComp
 $Comp
-L Custom_Schematic_Library:CY8C4245AZI-M433(48_TQPF) MP2
+L Custom_Schematic_Library:CY8C4245AZI-M433(48_TQPF) MUX2
 U 1 1 5DAF5D07
 P 17100 11350
-F 0 "MP2" H 17100 11250 50  0000 C CNN
+F 0 "MUX2" H 17100 11250 50  0000 C CNN
 F 1 "CY8C4245AZI-M433(48_TQPF)" H 17100 11500 50  0000 C CNN
 F 2 "Package_QFP:TQFP-48_7x7mm_P0.5mm" H 17100 11350 50  0001 C CNN
@@
 $EndComp
 $Comp
-L Custom_Schematic_Library:CY8C4245AZI-M433(48_TQPF) MP3
+L Custom_Schematic_Library:CY8C4245AZI-M433(48_TQPF) MUX3
 U 1 1 5DB30235
 P 23700 17250
-F 0 "MP3" H 23700 17150 50  0000 C CNN
+F 0 "MUX3" H 23700 17150 50  0000 C CNN
 F 1 "CY8C4245AZI-M433(48_TQPF)" H 23700 17350 50  0000 C CNN
 F 2 "Package_QFP:TQFP-48_7x7mm_P0.5mm" H 23700 17250 50  0001 C CNN
@@
 $EndComp
 $Comp
-L Custom_Schematic_Library:CY8C4245AZI-M433(48_TQPF) MP4
+L Custom_Schematic_Library:CY8C4245AZI-M433(48_TQPF) MUX4
 U 1 1 5DB85BD2
 P 16850 17200
-F 0 "MP4" H 16850 17100 50  0000 C CNN
+F 0 "MUX4" H 16850 17100 50  0000 C CNN
 F 1 "CY8C4245AZI-M433(48_TQPF)" H 16850 17300 50  0000 C CNN
 F 2 "Package_QFP:TQFP-48_7x7mm_P0.5mm" H 16850 17200 50  0001 C CNN
