File: PCB Layouts/Layout 2_15/Selection Interface.sch (KiCad schematic (older format))
At the start: 132 parts, among them P1 CONN_01X02, P11 CONN_01X02, P12 CONN_01X02, P13 CONN_01X10, P14 CONN_01X02, P15 CONN_01X02, P16 CONN_01X02, P18 CONN_02X05, P2 CONN_01X02, P3 CONN_01X02, P4 CONN_01X02, P5 CONN_01X02, P6 CONN_02X10, P7 CONN_01X02, P8 CONN_02X04, P9 CONN_01X02

Commit message: Updated PCB schematic to use more standardized symbols and only symbols from a single custom schematic library (in the "lib" sub-folder). Trying to remove excess, irrelevant files that have been auto-generated over many design iterations
Parts:
- removed CPU1, CPU2: CY8C58_(100_TQFP), Package_QFP:TQFP-100_14x14mm_P0.5mm, symbol Selection-Interface-rescue:CY8C58_(100_TQFP)
- removed P13: CONN_01X10, Connector_PinHeader_2.54mm:PinHeader_1x10_P2.54mm_Vertical_SMD_Pin1Left, symbol Selection-Interface-rescue:CONN_01X10
- removed P18: CONN_02X05, Connector_PinHeader_2.54mm:PinHeader_2x05_P2.54mm_Vertical_SMD, symbol Selection-Interface-rescue:CONN_02X05
- removed P6: CONN_02X10, Connector_PinHeader_2.54mm:PinHeader_2x10_P2.54mm_Vertical_SMD, symbol Selection-Interface-rescue:CONN_02X10
- removed P8: CONN_02X04, Connector_PinHeader_2.54mm:PinHeader_2x04_P2.54mm_Vertical_SMD, symbol Selection-Interface-rescue:CONN_02X04
- removed SOCKET1: 68_PLCC_Socket_(8468-21B1-RK-TP), Custom_Footprint_Library:68_PLCC_Socket_(8468-21B1-RK-TP), symbol Selection-Interface-rescue:68_PLCC_Socket_(8468-21B1-RK-TP)
- removed USB1, USB2: USB_2.0_B, Custom_Footprint_Library:Micro_USB_2.0_B_SMD(10118192-0001LF), symbol Selection-Interface-rescue:USB_2.0_B
- added B1: Conn_02x04_Odd_Even, Connector_PinHeader_2.54mm:PinHeader_2x04_P2.54mm_Vertical_SMD, symbol Connector_Generic:Conn_02x04_Odd_Even
- added CPU1, CPU2: CY8C58_(100_TQFP), Package_QFP:TQFP-100_14x14mm_P0.5mm, symbol Custom_Schematic_Library:CY8C58_(100_TQFP)
- added DISP1: Conn_01x10, Connector_PinHeader_2.54mm:PinHeader_1x10_P2.54mm_Vertical_SMD_Pin1Left, symbol Connector_Generic:Conn_01x10
- added OUT1: Conn_02x10_Odd_Even, Connector_PinHeader_2.54mm:PinHeader_2x10_P2.54mm_Vertical_SMD, symbol Connector_Generic:Conn_02x10_Odd_Even
- added PROG1: Conn_02x05_Odd_Even, Connector_PinHeader_2.54mm:PinHeader_2x05_P2.54mm_Vertical_SMD, symbol Connector_Generic:Conn_02x05_Odd_Even
- added SOCKET1: 68_PLCC_Socket_(8468-21B1-RK-TP), Custom_Footprint_Library:68_PLCC_Socket_(8468-21B1-RK-TP), symbol Custom_Schematic_Library:68_PLCC_Socket_(8468-21B1-RK-TP)
- added USB1, USB2: USB_2.0_B, Custom_Footprint_Library:Micro_USB_2.0_B_SMD(10118192-0001LF), symbol Custom_Schematic_Library:USB_2.0_B
Connections:
- net labels added: BT1_RXR, BT2_RXR, USB1_D+, USB1_D-, USB1_ID, USB2_D+, USB2_D-, USB2_ID, USBDM_C1, USBDM_C2, USBDP_C1, USBDP_C2, VBUS1, VBUS2, VCCA_C1, VCCA_C2, VCCD_C1, VCCD_C2, VCCD_M1, VCCD_M2, VCCD_M3, VCCD_M4, VDDA_C1, VDDA_C2, VDDA_M1, VDDA_M2, VDDA_M3, VDDA_M4
- wire segments 282 -> 279
Other:
- note added: "- Don’t have gates permanently connected to PSoCs\n- Break out I2C\n- Give Masters ability to reset Slaves\n- Add more optional TIA resistors\n- Communication between Masters\n- Clock sync between Masters\n- Resistor dividers for input measurements (esp. from AFM)\n- Boost converter for larger gate drive on board\n- Add interface for external chip (tire sensors)\n- Add interface for non-packaged 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"
- note removed: "- Don’t have gates permanently connected to PSoCs\n- Break out I2C\n- Give Masters ability to reset Slaves\n- Add more optional TIA resistors\n- DONE: Give PSoCs more natural number labels\n- Communication between Masters\n- Clock sync between Masters\n- Resistor dividers for input measurements (esp. from AFM)\n- Boost converter for larger gate drive on board\n- Add interface for external chip (t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"
