File: PCB Layouts/Layout 2_18/Selection Interface.sch (KiCad schematic (older format))
At the start: 132 parts

Commit message: Removed display header from layout 2_18
Parts:
- removed DISP1: Conn_01x10, Connector_PinHeader_2.54mm:PinHeader_1x10_P2.54mm_Vertical_SMD_Pin1Left, symbol Connector_Generic:Conn_01x10
Connections:
- net labels removed: CardCS, DisplayCS, DisplayDataOrCommand, DisplayMISO, DisplayMOSI, DisplayReset, DisplaySCK
Changed lines of the file:
@@
 Text GLabel 3700 1550 2    39   Input ~ 0
-VDDD
-Text GLabel 5600 4100 0    39   Input ~ 0
-DisplayMISO
-Text GLabel 5600 4200 0    39   Input ~ 0
-DisplaySCK
-Text GLabel 5600 4300 0    39   Input ~ 0
-DisplayMOSI
-Text GLabel 5600 4400 0    39   Input ~ 0
-DisplayCS
-Text GLabel 5600 4500 0    39   Input ~ 0
-CardCS
-Text GLabel 5600 4600 0    39   Input ~ 0
-DisplayDataOrCommand
-Text GLabel 5600 4700 0    39   Input ~ 0
-DisplayReset
-Text GLabel 5600 4800 0    39   Input ~ 0
-VDDD
-Text GLabel 5600 4900 0    39   Input ~ 0
-GND
-Text GLabel 15250 1300 0    39   Input ~ 0
-DisplayMISO
-Text GLabel 15250 1400 0    39   Input ~ 0
-DisplaySCK
-Text GLabel 15250 1500 0    39   Input ~ 0
-DisplayMOSI
-Text GLabel 15250 1800 0    39   Input ~ 0
-DisplayCS
-Text GLabel 15250 1900 0    39   Input ~ 0
-CardCS
-Text GLabel 15250 2000 0    39   Input ~ 0
-DisplayDataOrCommand
-Text GLabel 15250 2100 0    39   Input ~ 0
-DisplayReset
-Text GLabel 5600 4000 0    39   Input ~ 0
 VDDD
 Text GLabel 7300 4600 0    39   Input ~ 0
@@
 	1    0    0    -1
 $EndComp
-$Comp
-L Connector_Generic:Conn_01x10 DISP1
-U 1 1 5DB692F1
-P 5800 4400
-F 0 "DISP1" H 5800 4900 50  0000 C CNN
-F 1 "Conn_01x10" V 5900 4400 50  0000 C CNN
-F 2 "Connector_PinHeader_2.54mm:PinHeader_1x10_P2.54mm_Vertical_SMD_Pin1Left" H 5800 4400 50  0001 C CNN
-F 3 "~" H 5800 4400 50  0001 C CNN
-	1    5800 4400
-	1    0    0    -1
-$EndComp

Commit message: Removed secondary master processor (CPU2) from Layout 2_18
Parts:
- removed C1, C2, C3, C4, C64, C65, C68, C73, C74: 0.1uF, Capacitor_SMD:C_0603_1608Metric, symbol Device:C
- removed C60, C61, C66, C69, C70: 47uF, Capacitor_SMD:C_0603_1608Metric, symbol Device:C
- removed C62, C63, C67, C71, C72: 1uF, Capacitor_SMD:C_0603_1608Metric, symbol Device:C
- removed CPU2: CY8C58_(100_TQFP), Package_QFP:TQFP-100_14x14mm_P0.5mm, symbol Custom_Schematic_Library:CY8C58_(100_TQFP)
- removed FB7, FB8, R11, R12, R13, R14: R, Resistor_SMD:R_0603_1608Metric, symbol Device:R
- removed R10, R9: 22R, Resistor_SMD:R_0603_1608Metric, symbol Device:R
- removed R17: 1k, Resistor_SMD:R_0603_1608Metric, symbol Device:R
- removed R18: 2k, Resistor_SMD:R_0603_1608Metric, symbol Device:R
- removed USB2: USB_2.0_B, Custom_Footprint_Library:Micro_USB_2.0_B_SMD(10118192-0001LF), symbol Custom_Schematic_Library:USB_2.0_B
Connections:
- net labels removed: BT2_RX, BT2_RXR, BT2_TX, SWDCLK6, SWDIO6, USB2_D+, USB2_D-, USB2_ID, USBDM_C2, USBDP_C2, VBUS2, VCCA_C2, VCCD_C2, VDDA_C2
- wire segments 276 -> 196
Other:
- note added: "- Break out I2C\n- Give Masters ability to reset Slaves\n- PROGRESS: Add more optional TIA resistors\n- Resistor dividers for input measurements (esp. from AFM)\n- Boost converter for larger gate drive on board\n- Add interface for external chip (tire sensors)\n- Add interface for non-packaged chip (pogo pins)\n- Add temperature, humidity, and pressure sensors\n"
- note removed: "- Break out I2C\n- Give Masters ability to reset Slaves\n- PROGRESS: Add more optional TIA resistors\n- Communication between Masters\n- Clock sync between Masters\n- Resistor dividers for input measurements (esp. from AFM)\n- Boost converter for larger gate drive on board\n- Add interface for external chip (tire sensors)\n- Add interface for non-packaged chip (pogo pins)\n- Add temperature, humi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"

Commit message: Removed four IPEX connectors (for all of the miscellaneous IO pins). Also moved the bluetooth connector much closer to the microcontroller
Parts:
- removed IPEX10, IPEX11, IPEX12, IPEX9: Conn_01x02, Custom_Footprint_Library:IPEX_Connector_SMD_(RECE.20279.001E.01), symbol Connector_Generic:Conn_01x02
Connections:
- net labels removed: I2, I3, I4, I5, I6, I7, I8
Changed lines of the file:
@@
 Text GLabel 10200 2050 2    39   Input ~ 0
 GND_GPIO
-Text GLabel 10250 2500 0    39   Input ~ 0
-I2
-Text GLabel 10250 2600 0    39   Input ~ 0
-I3
-Text GLabel 10250 2700 0    39   Input ~ 0
-I4
-Text GLabel 10250 2800 0    39   Input ~ 0
-I5
-Text GLabel 10250 2900 0    39   Input ~ 0
-I6
-Text GLabel 10250 3000 0    39   Input ~ 0
-I7
-Text GLabel 10350 2800 2    39   Input ~ 0
-SS2
 Text GLabel 9700 2050 0    39   Input ~ 0
 GND
-Text GLabel 10350 2500 2    39   Input ~ 0
-SolutionGate
-Text GLabel 10350 2600 2    39   Input ~ 0
-LocalGates
-Text GLabel 10350 2700 2    39   Input ~ 0
-BackGate
-Text GLabel 10350 2900 2    39   Input ~ 0
-SS1
-Text GLabel 10350 3000 2    39   Input ~ 0
-DD2
 Text GLabel 19800 3200 2    39   Input ~ 0
 IO2
@@
 Text GLabel 6300 5800 1    39   Input ~ 0
 DD1
-Text GLabel 6800 5800 1    39   Input ~ 0
-IO1
-Text GLabel 7300 5800 1    39   Input ~ 0
-IO2
-Text GLabel 7800 5800 1    39   Input ~ 0
-IO3
-Text GLabel 8300 5800 1    39   Input ~ 0
-IO4
 Text GLabel 25100 11000 2    39   Input ~ 0
 XRES
@@
 	1    0    0    -1
 $EndComp
-Text GLabel 10250 3100 0    39   Input ~ 0
-I8
-Text GLabel 10350 3100 2    39   Input ~ 0
-DD1
 Text GLabel 19800 1800 2    39   Input ~ 0
 IO3
@@
 	0    1    1    0
 $EndComp
-$Comp
-L Connector_Generic:Conn_01x02 IPEX9
-U 1 1 5DB22D42
-P 6800 6000
-F 0 "IPEX9" V 6900 5950 50  0000 C CNN
-F 1 "Conn_01x02" V 7000 5950 50  0000 C CNN
-F 2 "Custom_Footprint_Library:IPEX_Connector_SMD_(RECE.20279.001E.01)" H 6800 6000 50  0001 C CNN
-F 3 "~" H 6800 6000 50  0001 C CNN
-	1    6800 6000
-	0    1    1    0
-$EndComp
-$Comp
-L Connector_Generic:Conn_01x02 IPEX10
-U 1 1 5DB22EDB
-P 7300 6000
-F 0 "IPEX10" V 7400 5950 50  0000 C CNN
-F 1 "Conn_01x02" V 7500 5950 50  0000 C CNN
-F 2 "Custom_Footprint_Library:IPEX_Connector_SMD_(RECE.20279.001E.01)" H 7300 6000 50  0001 C CNN
-F 3 "~" H 7300 6000 50  0001 C CNN
-	1    7300 6000
-	0    1    1    0
-$EndComp
-$Comp
-L Connector_Generic:Conn_01x02 IPEX11
-U 1 1 5DB23078
-P 7800 6000
-F 0 "IPEX11" V 7900 5950 50  0000 C CNN
-F 1 "Conn_01x02" V 8000 5950 50  0000 C CNN
-F 2 "Custom_Footprint_Library:IPEX_Connector_SMD_(RECE.20279.001E.01)" H 7800 6000 50  0001 C CNN
-F 3 "~" H 7800 6000 50  0001 C CNN
-	1    7800 6000
-	0    1    1    0
-$EndComp
-$Comp
-L Connector_Generic:Conn_01x02 IPEX12
-U 1 1 5DB23219
-P 8300 6000
-F 0 "IPEX12" V 8400 5950 50  0000 C CNN
-F 1 "Conn_01x02" V 8500 5950 50  0000 C CNN
-F 2 "Custom_Footprint_Library:IPEX_Connector_SMD_(RECE.20279.001E.01)" H 8300 6000 50  0001 C CNN
-F 3 "~" H 8300 6000 50  0001 C CNN
-	1    8300 6000
-	0    1    1    0
-$EndComp

Commit message: Removed the IPEX connection for GND, and got rid of some extra pins on the PROG2 header
Parts:
- removed IPEX1: Conn_01x02, Custom_Footprint_Library:IPEX_Connector_SMD_(RECE.20279.001E.01), symbol Connector_Generic:Conn_01x02
- removed PROG2: Conn_02x06_Odd_Even, Connector_PinHeader_2.54mm:PinHeader_2x06_P2.54mm_Vertical_SMD, symbol Connector_Generic:Conn_02x06_Odd_Even
- added PROG2: Conn_02x05_Odd_Even, Connector_PinHeader_2.54mm:PinHeader_2x05_P2.54mm_Vertical_SMD, symbol Connector_Generic:Conn_02x05_Odd_Even
Changed lines of the file:
@@
 Text GLabel 7300 4900 0    39   Input ~ 0
 IO4
-Text GLabel 2800 5800 1    39   Input ~ 0
-GND_GPIO
 Text GLabel 3300 5800 1    39   Input ~ 0
 SolutionGate_Socket
@@
 Text GLabel 19800 1800 2    39   Input ~ 0
 IO3
-$Comp
-L Connector_Generic:Conn_02x06_Odd_Even PROG2
-U 1 1 5DA1458B
-P 3300 4600
-F 0 "PROG2" H 3350 5017 50  0000 C CNN
-F 1 "Conn_02x06_Odd_Even" H 3350 4926 50  0000 C CNN
-F 2 "Connector_PinHeader_2.54mm:PinHeader_2x06_P2.54mm_Vertical_SMD" H 3300 4600 50  0001 C CNN
-F 3 "~" H 3300 4600 50  0001 C CNN
-	1    3300 4600
-	1    0    0    -1
-$EndComp
 Text GLabel 3100 4400 0    50   Input ~ 0
 SWDCLK1
@@
 	17600 3500 17600 4200
 $Comp
-L Connector_Generic:Conn_01x02 IPEX1
-U 1 1 5DB20476
-P 2800 6000
-F 0 "IPEX1" V 2900 5950 50  0000 C CNN
-F 1 "Conn_01x02" V 3000 5950 50  0000 C CNN
-F 2 "Custom_Footprint_Library:IPEX_Connector_SMD_(RECE.20279.001E.01)" H 2800 6000 50  0001 C CNN
-F 3 "~" H 2800 6000 50  0001 C CNN
-	1    2800 6000
-	0    1    1    0
-$EndComp
-$Comp
 L Connector_Generic:Conn_01x02 IPEX2
 U 1 1 5DB21D81
@@
 Text GLabel 7300 4300 0    39   Input ~ 0
 GND
+$Comp
+L Connector_Generic:Conn_02x05_Odd_Even PROG2
+U 1 1 5DC89FB3
+P 3300 4600
+F 0 "PROG2" H 3350 5017 50  0000 C CNN
+F 1 "Conn_02x05_Odd_Even" H 3350 4926 50  0000 C CNN
+F 2 "Connector_PinHeader_2.54mm:PinHeader_2x05_P2.54mm_Vertical_SMD" H 3300 4600 50  0001 C CNN
+F 3 "~" H 3300 4600 50  0001 C CNN
+	1    3300 4600
+	1    0    0    -1
+$EndComp
 $EndSCHEMATC

Commit message: Finished moving CPU1 and re-connecting all signals. Started arranging external resistors and moved bluetooth connector even closer
Parts:
- R5: value R -> 100M
- R6, R8: value R -> 1M
- R7: value R -> 10k
Connections:
- net labels added: Gate_R1M_High, Gate_R1M_Low, OPAMP_VOUT, OPAMP_Vminus, OPAMP_Vplus, TIA_R100M, TIA_R10k, TIA_R1M, TIA_R_COMMON
- wire segments 196 -> 198
Changed lines of the file:
@@
 VSSD
-Wire Wire Line
-	15250 2700 14650 2700
-Wire Wire Line
-	14650 2700 14650 3400
 Wire Wire Line
 	15250 3200 14450 3200
 Wire Wire Line
 	15250 3300 14450 3300
-Wire Wire Line
-	14650 3400 14450 3400
 Wire Wire Line
 	23250 13000 23250 12600
@@
 L Device:R R7
 U 1 1 599FA581
-P 18300 650
-F 0 "R7" V 18380 650 50  0000 C CNN
-F 1 "R" V 18300 650 50  0000 C CNN
-F 2 "Resistor_SMD:R_0603_1608Metric" V 18230 650 50  0001 C CNN
-F 3 "" H 18300 650 50  0000 C CNN
-	1    18300 650
-	1    0    0    -1
-$EndComp
-$Comp
-L Device:R R5
-U 1 1 599FA76F
-P 17900 650
-F 0 "R5" V 17980 650 50  0000 C CNN
-F 1 "R" V 17900 650 50  0000 C CNN
-F 2 "Resistor_SMD:R_0603_1608Metric" V 17830 650 50  0001 C CNN
-F 3 "" H 17900 650 50  0000 C CNN
-	1    17900 650
-	1    0    0    -1
+P 18300 -350
+F 0 "R7" V 18380 -350 50  0000 C CNN
+F 1 "10k" V 18300 -350 50  0000 C CNN
+F 2 "Resistor_SMD:R_0603_1608Metric" V 18230 -350 50  0001 C CNN
+F 3 "" H 18300 -350 50  0000 C CNN
+	1    18300 -350
+	-1   0    0    1
 $EndComp
 $Comp
 L Device:R R6
 U 1 1 599FA901
-P 18100 650
-F 0 "R6" V 18180 650 50  0000 C CNN
-F 1 "R" V 18100 650 50  0000 C CNN
-F 2 "Resistor_SMD:R_0603_1608Metric" V 18030 650 50  0001 C CNN
-F 3 "" H 18100 650 50  0000 C CNN
-	1    18100 650
-	1    0    0    -1
+P 18000 -50
+F 0 "R6" V 18080 -50 50  0000 C CNN
+F 1 "1M" V 18000 -50 50  0000 C CNN
+F 2 "Resistor_SMD:R_0603_1608Metric" V 17930 -50 50  0001 C CNN
+F 3 "" H 18000 -50 50  0000 C CNN
+	1    18000 -50
+	-1   0    0    1
 $EndComp
 $Comp
 L Device:R R8
 U 1 1 599FAA80
-P 18500 650
-F 0 "R8" V 18580 650 50  0000 C CNN
-F 1 "R" V 18500 650 50  0000 C CNN
-F 2 "Resistor_SMD:R_0603_1608Metric" V 18430 650 50  0001 C CNN
-F 3 "" H 18500 650 50  0000 C CNN
-	1    18500 650
-	1    0    0    -1
-$EndComp
-Wire Wire Line
-	17900 500  18000 500
-Wire Wire Line
-	18000 500  18000 800
-Wire Wire Line
-	18100 500  18200 500
-Wire Wire Line
-	18200 500  18200 800
-Wire Wire Line
-	18300 500  18400 500
-Wire Wire Line
-	18400 500  18400 800
-Wire Wire Line
-	18500 500  18600 500
-Wire Wire Line
-	18600 500  18600 800
+P 14550 1800
+F 0 "R8" V 14630 1800 50  0000 C CNN
+F 1 "1M" V 14550 1800 50  0000 C CNN
+F 2 "Resistor_SMD:R_0603_1608Metric" V 14480 1800 50  0001 C CNN
+F 3 "" H 14550 1800 50  0000 C CNN
+	1    14550 1800
+	0    1    1    0
+$EndComp
 Text GLabel 9700 1900 0    39   Input ~ 0
 GND
@@
 Text GLabel 14450 3300 0    39   Input ~ 0
 SWDCLK5
-Text GLabel 14450 3400 0    39   Input ~ 0
+Text GLabel 14450 2700 0    39   Input ~ 0
 XRES
 Text GLabel 3600 3600 2    39   Input ~ 0
@@
 	1    0    0    -1
 $EndComp
+Wire Wire Line
+	14450 2700 15250 2700
+Wire Wire Line
+	18300 -500 18200 -500
+Text GLabel 18200 -500 1    39   Input ~ 0
+TIA_R_COMMON
+Text GLabel 18100 800  1    39   Input ~ 0
+TIA_R100M
+Text GLabel 18000 800  1    39   Input ~ 0
+TIA_R1M
+Text GLabel 18300 800  1    39   Input ~ 0
+TIA_R10k
+$Comp
+L Device:R R5
+U 1 1 599FA76F
+P 18100 250
+F 0 "R5" V 18180 250 50  0000 C CNN
+F 1 "100M" V 18100 250 50  0000 C CNN
+F 2 "Resistor_SMD:R_0603_1608Metric" V 18030 250 50  0001 C CNN
+F 3 "" H 18100 250 50  0000 C CNN
+	1    18100 250
+	-1   0    0    1
+$EndComp
+Wire Wire Line
+	18300 -200 18300 800
+Wire Wire Line
+	18000 100  18000 800
+Wire Wire Line
+	18100 400  18100 800
+Text GLabel 15250 1900 0    39   Input ~ 0
+Gate_R1M_High
+Text GLabel 15250 1800 0    39   Input ~ 0
+Gate_R1M_Low
+Wire Wire Line
+	14700 1800 15250 1800
+Wire Wire Line
+	14400 1800 14400 1900
+Wire Wire Line
+	14400 1900 15250 1900
+Wire Wire Line
+	18000 -200 18200 -200
+Wire Wire Line
+	18200 -200 18200 100
+Wire Wire Line
+	18100 100  18200 100
+Connection ~ 18200 100
+Wire Wire Line
+	18200 100  18200 800
+Wire Wire Line
+	18200 -200 18200 -500
+Connection ~ 18200 -200
+Text GLabel 15250 2800 0    39   Input ~ 0
+OPAMP_VOUT
+Text GLabel 15250 2100 0    39   Input ~ 0
+OPAMP_Vplus
+Text GLabel 15250 2000 0    39   Input ~ 0
+OPAMP_Vminus
 $EndSCHEMATC

Commit message: Added external op-amp schematic and footprint. Continuing to make progress in slimming down the PCB
Parts:
- removed C7: 0.1uF, Capacitor_SMD:C_0603_1608Metric, symbol Device:C
- added AMP1: OPA363, Package_TO_SOT_SMD:SOT-23-6, symbol Custom_Schematic_Library:OPA363
- added C60: 1pF, Capacitor_SMD:C_0603_1608Metric, symbol Device:C
Connections:
- net labels added: AMP1_VOUT, AMP1_Vminus, AMP1_Vplus
- net labels removed: OPAMP_VOUT, OPAMP_Vminus, OPAMP_Vplus
- wire segments 198 -> 209
Changed lines of the file:
@@
 Text GLabel 17150 0    2    39   Input ~ 0
-VSSD
-Text GLabel 17150 500  2    39   Input ~ 0
 VSSD
 $Comp
@@
 $EndComp
 $Comp
-L Device:C C7
-U 1 1 599D66A9
-P 10150 1000
-F 0 "C7" H 10175 1100 50  0000 L CNN
-F 1 "0.1uF" H 10175 900 50  0000 L CNN
-F 2 "Capacitor_SMD:C_0603_1608Metric" H 10188 850 50  0001 C CNN
-F 3 "" H 10150 1000 50  0000 C CNN
-	1    10150 1000
-	1    0    0    1
-$EndComp
-$Comp
 L Device:C C8
 U 1 1 599D675F
@@
 $EndComp
 Connection ~ 9850 850
-Connection ~ 10150 850
 Connection ~ 10450 850
 Connection ~ 9850 1150
-Connection ~ 10150 1150
 Connection ~ 10450 1150
 Text GLabel 10750 1150 2    39   Input ~ 0
@@
 	9550 850  9850 850
 Wire Wire Line
-	9850 850  10150 850
-Wire Wire Line
-	10150 850  10450 850
-Wire Wire Line
 	10450 850  10750 850
 Wire Wire Line
 	9550 1150 9850 1150
-Wire Wire Line
-	9850 1150 10150 1150
-Wire Wire Line
-	10150 1150 10450 1150
 Wire Wire Line
 	10450 1150 10750 1150
@@
 	18200 -200 18200 -500
 Connection ~ 18200 -200
-Text GLabel 15250 2800 0    39   Input ~ 0
-OPAMP_VOUT
-Text GLabel 15250 2100 0    39   Input ~ 0
-OPAMP_Vplus
-Text GLabel 15250 2000 0    39   Input ~ 0
-OPAMP_Vminus
+Text GLabel 16800 -1300 0    39   Input ~ 0
+AMP1_VOUT
+Text GLabel 16800 -1100 0    39   Input ~ 0
+AMP1_Vplus
+Text GLabel 17600 -1100 2    39   Input ~ 0
+AMP1_Vminus
+$Comp
+L Custom_Schematic_Library:OPA363 AMP1
+U 1 1 5DB59C43
+P 17200 -1200
+F 0 "AMP1" H 17200 -835 50  0000 C CNN
+F 1 "OPA363" H 17200 -926 50  0000 C CNN
+F 2 "Package_TO_SOT_SMD:SOT-23-6" H 17200 -750 50  0001 C CNN
+F 3 "" H 17200 -750 50  0001 C CNN
+	1    17200 -1200
+	1    0    0    -1
+$EndComp
+Text GLabel 17600 -1300 2    39   Input ~ 0
+VDDD
+Text GLabel 16800 -1200 0    39   Input ~ 0
+GND
+Wire Wire Line
+	17600 -1200 17600 -1300
+Wire Wire Line
+	17600 -1100 17900 -1100
+Wire Wire Line
+	16800 -950 16800 -1100
+$Comp
+L Device:C C60
+U 1 1 5DC4A0EA
+P 17750 -950
+F 0 "C60" H 17775 -850 50  0000 L CNN
+F 1 "1pF" H 17775 -1050 50  0000 L CNN
+F 2 "Capacitor_SMD:C_0603_1608Metric" H 17788 -1100 50  0001 C CNN
+F 3 "" H 17750 -950 50  0000 C CNN
+	1    17750 -950
+	0    1    1    0
+$EndComp
+Wire Wire Line
+	17600 -950 16800 -950
+Wire Wire Line
+	17600 -950 17600 -700
+Wire Wire Line
+	17600 -700 17800 -700
+Wire Wire Line
+	17800 -700 17800 800
+Wire Wire Line
+	17900 -1100 17900 -950
+Connection ~ 17900 -950
+Wire Wire Line
+	17900 -950 17900 800
+Connection ~ 17600 -950
+Wire Wire Line
+	16600 800  16600 550
+Wire Wire Line
+	16600 550  16150 550
+Wire Wire Line
+	16150 550  16150 -1300
+Wire Wire Line
+	16150 -1300 16800 -1300
+Wire Wire Line
+	9850 1150 10450 1150
+Wire Wire Line
+	9850 850  10450 850
+Text GLabel 17150 500  2    39   Input ~ 0
+VSSD
 $EndSCHEMATC

Commit message: Converted all CPU gate channels to a single CPU gate channel. Also continued shrinking and cleaning up routing
Connections:
- net labels added: Gate
- net labels removed: BackGate, LocalGates, SolutionGate
Changed lines of the file:
@@
 GND_GPIO
 Text GLabel 15250 3700 0    39   Input ~ 0
-SolutionGate
-Text GLabel 16500 4200 3    39   Input ~ 0
-LocalGates
-Text GLabel 16800 4200 3    39   Input ~ 0
-BackGate
+Gate
 Text GLabel 17000 4200 3    39   Input ~ 0
 IO1
@@
 DD1
 Text GLabel 7300 4100 0    39   Input ~ 0
-LocalGates
+Gate
 Text GLabel 7800 4300 2    39   Input ~ 0
 GND
 Text GLabel 7300 4200 0    39   Input ~ 0
-BackGate
+Gate
 Text GLabel 7300 4000 0    39   Input ~ 0
-SolutionGate
+Gate
 Text GLabel 10200 2050 2    39   Input ~ 0
 GND_GPIO

Commit message: Starting to put on the finishing touches to Layout 2_18
Other:
- note added: "- Break out I2C\n- Give Masters ability to reset Slaves\n- Resistor dividers for input measurements (esp. from AFM)\n- Boost converter for larger gate drive on board\n- Add interface for external chip (tire sensors)\n- Add interface for non-packaged chip (pogo pins)\n- Add temperature, humidity, and pressure sensors\n"
- note removed: "- Break out I2C\n- Give Masters ability to reset Slaves\n- PROGRESS: Add more optional TIA resistors\n- Resistor dividers for input measurements (esp. from AFM)\n- Boost converter for larger gate drive on board\n- Add interface for external chip (tire sensors)\n- Add interface for non-packaged chip (pogo pins)\n- Add temperature, humidity, and pressure sensors\n"
Changed lines of the file:
@@
 GND
 Text Notes 2550 7500 0    60   ~ 0
-- Break out I2C\n- Give Masters ability to reset Slaves\n- PROGRESS: Add more optional TIA resistors\n- Resistor dividers for input measurements (esp. from AFM)\n- Boost converter for larger gate drive on board\n- Add interface for external chip (tire sensors)\n- Add interface for non-packaged chip (pogo pins)\n- Add temperature, humidity, and pressure sensors\n
+- Break out I2C\n- Give Masters ability to reset Slaves\n- Resistor dividers for input measurements (esp. from AFM)\n- Boost converter for larger gate drive on board\n- Add interface for external chip (tire sensors)\n- Add interface for non-packaged chip (pogo pins)\n- Add temperature, humidity, and pressure sensors\n
 Wire Wire Line
 	20900 2600 21350 2600
