File: PCB Layouts/Layout 2_19/Selection Interface.sch (KiCad schematic (older format))
At the start: 87 parts

Commit message: Updated recommended value of CG1 in Layout 2_19 based on my tests this afternoon
Parts:
- CG1: value 1uF -> 1nF
Changed lines of the file:
@@
 P 9900 5850
 F 0 "CG1" H 9925 5950 50  0000 L CNN
-F 1 "1uF" H 9925 5750 50  0000 L CNN
+F 1 "1nF" H 9925 5750 50  0000 L CNN
 F 2 "Capacitor_SMD:C_0603_1608Metric" H 9938 5700 50  0001 C CNN
 F 3 "" H 9900 5850 50  0000 C CNN

Commit message: Slight tweaks to Layout 2_19 (removed unnecessary Gate capacitor, compressed some BT signal wiring)
Parts:
- removed CG1: 1nF, Capacitor_SMD:C_0603_1608Metric, symbol Device:C
Changed lines of the file:
@@
 Wire Wire Line
 	17450 9200 18700 9200
-$Comp
-L Device:C CG1
-U 1 1 5DE5749E
-P 9900 5850
-F 0 "CG1" H 9925 5950 50  0000 L CNN
-F 1 "1nF" H 9925 5750 50  0000 L CNN
-F 2 "Capacitor_SMD:C_0603_1608Metric" H 9938 5700 50  0001 C CNN
-F 3 "" H 9900 5850 50  0000 C CNN
-	1    9900 5850
-	1    0    0    -1
-$EndComp
-Text GLabel 9900 5700 1    39   Input ~ 0
-Gate
-Text GLabel 9900 6000 3    39   Input ~ 0
-GND
 $EndSCHEMATC

Commit message: In Layout 2_19, added SMD capacitor for the gate signal
Parts:
- added CG1: 1uF, Capacitor_SMD:C_0603_1608Metric, symbol Device:C
Changed lines of the file:
@@
 Wire Wire Line
 	17450 9200 18700 9200
+$Comp
+L Device:C CG1
+U 1 1 5DE5749E
+P 9900 5850
+F 0 "CG1" H 9925 5950 50  0000 L CNN
+F 1 "1uF" H 9925 5750 50  0000 L CNN
+F 2 "Capacitor_SMD:C_0603_1608Metric" H 9938 5700 50  0001 C CNN
+F 3 "" H 9900 5850 50  0000 C CNN
+	1    9900 5850
+	1    0    0    -1
+$EndComp
+Text GLabel 9900 5700 1    39   Input ~ 0
+Gate
+Text GLabel 9900 6000 3    39   Input ~ 0
+GND
 $EndSCHEMATC
