File: PCB Layouts/Layout 2_19/Selection Interface.sch (KiCad schematic (older format))
At the start: 97 parts, among them J1 Conn_01x02

Commit message: Decided to make connection between TIA_R_Common and op-amp Vout permanent to reduce solder complexity and because that pin cannot be routed by the PSoC anyway
Parts:
- removed J1: Conn_01x02, Jumper:SolderJumper-2_P1.3mm_Open_RoundedPad1.0x1.5mm, symbol Connector_Generic:Conn_01x02
Connections:
- net labels removed: TIA_R_COMMON
- wire segments 214 -> 211
Changed lines of the file:
@@
 Wire Wire Line
 	18300 -500 18200 -500
-Text GLabel 18200 -500 1    39   Input ~ 0
-TIA_R_COMMON
 Text GLabel 18100 800  1    39   Input ~ 0
 TIA_R100M
@@
 Wire Wire Line
 	18100 100  18200 100
-Connection ~ 18200 100
-Wire Wire Line
-	18200 100  18200 800
 Wire Wire Line
 	18200 -200 18200 -500
@@
 Text GLabel 17150 500  2    39   Input ~ 0
 VSSD
-$Comp
-L Connector_Generic:Conn_01x02 J1
-U 1 1 5DD45C60
-P 18200 -1700
-F 0 "J1" H 18280 -1708 50  0000 L CNN
-F 1 "Conn_01x02" H 18280 -1799 50  0000 L CNN
-F 2 "Jumper:SolderJumper-2_P1.3mm_Open_RoundedPad1.0x1.5mm" H 18200 -1700 50  0001 C CNN
-F 3 "~" H 18200 -1700 50  0001 C CNN
-	1    18200 -1700
-	1    0    0    -1
-$EndComp
 Wire Wire Line
 	16150 -1300 16150 -1700
+Connection ~ 16150 -1300
+Connection ~ 18200 -500
 Wire Wire Line
-	16150 -1700 18000 -1700
-Connection ~ 16150 -1300
+	18200 -1700 18200 -500
 Wire Wire Line
-	18000 -1600 18000 -1350
-Wire Wire Line
-	18000 -1350 18200 -1350
-Wire Wire Line
-	18200 -1350 18200 -500
-Connection ~ 18200 -500
+	16150 -1700 18200 -1700
 $EndSCHEMATC

Commit message: Added physical SAR bypass capacitor to Layout 2_19
Parts:
- added CB1: 1uF, Capacitor_SMD:C_0603_1608Metric, symbol Device:C
Connections:
- net labels added: DeltaSigma_Bypass_Cap, SAR1_Bypass_Cap, SAR2_Bypass_Cap
- wire segments 211 -> 213
Changed lines of the file:
@@
 	1    0    0    -1
 $EndComp
-$Comp
-L Custom_Schematic_Library:CY8C58_(100_TQFP) CPU1
-U 1 1 5DC0AF8F
-P 17500 2500
-F 0 "CPU1" H 17500 2300 50  0000 C CNN
-F 1 "CY8C58_(100_TQFP)" H 17500 2700 50  0000 C CNN
-F 2 "Package_QFP:TQFP-100_14x14mm_P0.5mm" H 17500 3000 50  0001 C CNN
-F 3 "DOCUMENTATION" H 17500 2100 50  0001 C CNN
-	1    17500 2500
-	1    0    0    -1
-$EndComp
-Wire Wire Line
-	17700 -300 17700 800
-Connection ~ 17700 800
-Wire Wire Line
-	17700 800  17700 3500
 Wire Wire Line
 	17600 3500 17600 4200
@@
 Wire Wire Line
 	16150 -1700 18200 -1700
+Text GLabel 18700 800  1    39   Input ~ 0
+SAR1_Bypass_Cap
+Text GLabel 19800 1500 2    39   Input ~ 0
+SAR2_Bypass_Cap
+Text GLabel 19800 1400 2    39   Input ~ 0
+DeltaSigma_Bypass_Cap
+Wire Wire Line
+	17700 800  17700 3500
+Wire Wire Line
+	17700 -300 17700 800
+Connection ~ 17700 800
+$Comp
+L Custom_Schematic_Library:CY8C58_(100_TQFP) CPU1
+U 1 1 5DC0AF8F
+P 17500 2500
+F 0 "CPU1" H 17500 2300 50  0000 C CNN
+F 1 "CY8C58_(100_TQFP)" H 17500 2700 50  0000 C CNN
+F 2 "Package_QFP:TQFP-100_14x14mm_P0.5mm" H 17500 3000 50  0001 C CNN
+F 3 "DOCUMENTATION" H 17500 2100 50  0001 C CNN
+	1    17500 2500
+	1    0    0    -1
+$EndComp
+$Comp
+L Device:C CB1
+U 1 1 5DDECF0D
+P 18700 0
+F 0 "CB1" H 18725 100 50  0000 L CNN
+F 1 "1uF" H 18725 -100 50  0000 L CNN
+F 2 "Capacitor_SMD:C_0603_1608Metric" H 18738 -150 50  0001 C CNN
+F 3 "" H 18700 0   50  0000 C CNN
+	1    18700 0
+	1    0    0    -1
+$EndComp
+Wire Wire Line
+	18700 150  18700 800
+Text GLabel 18700 -150 1    39   Input ~ 0
+VSSD
+Text GLabel 19450 500  0    39   Input ~ 0
+SAR1_Bypass_Cap
+Text GLabel 19650 500  2    39   Input ~ 0
+SAR2_Bypass_Cap
+Wire Wire Line
+	19450 500  19650 500
 $EndSCHEMATC

Commit message: Added a bypass capacitor for the delta-sigma ADC. Slightly improved the copper pours on a few layers
Parts:
- added CB2: 1uF, Capacitor_SMD:C_0603_1608Metric, symbol Device:C
Changed lines of the file:
@@
 Text GLabel 18700 -150 1    39   Input ~ 0
 VSSD
-Text GLabel 19450 500  0    39   Input ~ 0
-SAR1_Bypass_Cap
-Text GLabel 19650 500  2    39   Input ~ 0
-SAR2_Bypass_Cap
+$Comp
+L Device:C CB2
+U 1 1 5DDD7238
+P 20750 1400
+F 0 "CB2" H 20775 1500 50  0000 L CNN
+F 1 "1uF" H 20775 1300 50  0000 L CNN
+F 2 "Capacitor_SMD:C_0603_1608Metric" H 20788 1250 50  0001 C CNN
+F 3 "" H 20750 1400 50  0000 C CNN
+	1    20750 1400
+	0    1    1    0
+$EndComp
+Text GLabel 20900 1400 2    39   Input ~ 0
+VSSD
 Wire Wire Line
-	19450 500  19650 500
+	20600 1400 19800 1400
 $EndSCHEMATC

Commit message: Removed unused SMD capacitors from Layout 2_19
Parts:
- removed C17, C20, C43, C49: 47uF, Capacitor_SMD:C_0603_1608Metric, symbol Device:C
- removed C24, C27, C46, C55: 1uF, Capacitor_SMD:C_0603_1608Metric, symbol Device:C
- removed C31, C34, C52, C58: 0.1uF, Capacitor_SMD:C_0603_1608Metric, symbol Device:C
Connections:
- wire segments 213 -> 189
Changed lines of the file:
@@
-VSSD
-$Comp
-L Device:C C31
-U 1 1 599D2C02
-P 25050 9550
-F 0 "C31" H 25075 9650 50  0000 L CNN
-F 1 "0.1uF" H 25075 9450 50  0000 L CNN
-F 2 "Capacitor_SMD:C_0603_1608Metric" H 25088 9400 50  0001 C CNN
-F 3 "" H 25050 9550 50  0000 C CNN
-	1    25050 9550
-	1    0    0    -1
-$EndComp
-$Comp
-L Device:C C24
-U 1 1 599D2C08
-P 24750 9550
-F 0 "C24" H 24775 9650 50  0000 L CNN
-F 1 "1uF" H 24775 9450 50  0000 L CNN
-F 2 "Capacitor_SMD:C_0603_1608Metric" H 24788 9400 50  0001 C CNN
-F 3 "" H 24750 9550 50  0000 C CNN
-	1    24750 9550
-	1    0    0    -1
-$EndComp
-$Comp
-L Device:C C17
-U 1 1 599D2C0E
-P 24450 9550
-F 0 "C17" H 24475 9650 50  0000 L CNN
-F 1 "47uF" H 24475 9450 50  0000 L CNN
-F 2 "Capacitor_SMD:C_0603_1608Metric" H 24488 9400 50  0001 C CNN
-F 3 "" H 24450 9550 50  0000 C CNN
-	1    24450 9550
-	1    0    0    -1
-$EndComp
-Wire Wire Line
-	24450 9700 24750 9700
-Connection ~ 25050 9700
-Connection ~ 24750 9700
-Wire Wire Line
-	24050 9400 24450 9400
-Connection ~ 25050 9400
-Connection ~ 24750 9400
-Connection ~ 24450 9400
-Text GLabel 25300 9700 2    39   Input ~ 0
 VSSD
 $Comp
@@
 VSSD
 $Comp
-L Device:C C58
-U 1 1 599EBC64
-P 18450 9350
-F 0 "C58" H 18475 9450 50  0000 L CNN
-F 1 "0.1uF" H 18475 9250 50  0000 L CNN
-F 2 "Capacitor_SMD:C_0603_1608Metric" H 18488 9200 50  0001 C CNN
-F 3 "" H 18450 9350 50  0000 C CNN
-	1    18450 9350
-	1    0    0    -1
-$EndComp
-$Comp
-L Device:C C55
-U 1 1 599EBC6A
-P 18150 9350
-F 0 "C55" H 18175 9450 50  0000 L CNN
-F 1 "1uF" H 18175 9250 50  0000 L CNN
-F 2 "Capacitor_SMD:C_0603_1608Metric" H 18188 9200 50  0001 C CNN
-F 3 "" H 18150 9350 50  0000 C CNN
-	1    18150 9350
-	1    0    0    -1
-$EndComp
-$Comp
-L Device:C C49
-U 1 1 599EBC70
-P 17850 9350
-F 0 "C49" H 17875 9450 50  0000 L CNN
-F 1 "47uF" H 17875 9250 50  0000 L CNN
-F 2 "Capacitor_SMD:C_0603_1608Metric" H 17888 9200 50  0001 C CNN
-F 3 "" H 17850 9350 50  0000 C CNN
-	1    17850 9350
-	1    0    0    -1
-$EndComp
-Wire Wire Line
-	17850 9500 18150 9500
-Connection ~ 18450 9500
-Connection ~ 18150 9500
-Wire Wire Line
-	17450 9200 17850 9200
-Connection ~ 18450 9200
-Connection ~ 18150 9200
-Connection ~ 17850 9200
-Text GLabel 18700 9500 2    39   Input ~ 0
-VSSD
-$Comp
 L Device:C C57
 U 1 1 599EBC83
@@
 VSSD
 $Comp
-L Device:C C34
-U 1 1 599EC75C
-P 25050 15250
-F 0 "C34" H 25075 15350 50  0000 L CNN
-F 1 "0.1uF" H 25075 15150 50  0000 L CNN
-F 2 "Capacitor_SMD:C_0603_1608Metric" H 25088 15100 50  0001 C CNN
-F 3 "" H 25050 15250 50  0000 C CNN
-	1    25050 15250
-	1    0    0    -1
-$EndComp
-$Comp
-L Device:C C27
-U 1 1 599EC762
-P 24750 15250
-F 0 "C27" H 24775 15350 50  0000 L CNN
-F 1 "1uF" H 24775 15150 50  0000 L CNN
-F 2 "Capacitor_SMD:C_0603_1608Metric" H 24788 15100 50  0001 C CNN
-F 3 "" H 24750 15250 50  0000 C CNN
-	1    24750 15250
-	1    0    0    -1
-$EndComp
-$Comp
-L Device:C C20
-U 1 1 599EC768
-P 24450 15250
-F 0 "C20" H 24475 15350 50  0000 L CNN
-F 1 "47uF" H 24475 15150 50  0000 L CNN
-F 2 "Capacitor_SMD:C_0603_1608Metric" H 24488 15100 50  0001 C CNN
-F 3 "" H 24450 15250 50  0000 C CNN
-	1    24450 15250
-	1    0    0    -1
-$EndComp
-Wire Wire Line
-	24450 15400 24750 15400
-Connection ~ 25050 15400
-Connection ~ 24750 15400
-Wire Wire Line
-	24050 15100 24450 15100
-Connection ~ 25050 15100
-Connection ~ 24750 15100
-Connection ~ 24450 15100
-Text GLabel 25300 15400 2    39   Input ~ 0
-VSSD
-$Comp
 L Device:C C33
 U 1 1 599EC77B
@@
 VSSD
 $Comp
-L Device:C C52
-U 1 1 599F47F8
-P 18200 15200
-F 0 "C52" H 18225 15300 50  0000 L CNN
-F 1 "0.1uF" H 18225 15100 50  0000 L CNN
-F 2 "Capacitor_SMD:C_0603_1608Metric" H 18238 15050 50  0001 C CNN
-F 3 "" H 18200 15200 50  0000 C CNN
-	1    18200 15200
-	1    0    0    -1
-$EndComp
-$Comp
-L Device:C C46
-U 1 1 599F47FE
-P 17900 15200
-F 0 "C46" H 17925 15300 50  0000 L CNN
-F 1 "1uF" H 17925 15100 50  0000 L CNN
-F 2 "Capacitor_SMD:C_0603_1608Metric" H 17938 15050 50  0001 C CNN
-F 3 "" H 17900 15200 50  0000 C CNN
-	1    17900 15200
-	1    0    0    -1
-$EndComp
-$Comp
-L Device:C C43
-U 1 1 599F4804
-P 17600 15200
-F 0 "C43" H 17625 15300 50  0000 L CNN
-F 1 "47uF" H 17625 15100 50  0000 L CNN
-F 2 "Capacitor_SMD:C_0603_1608Metric" H 17638 15050 50  0001 C CNN
-F 3 "" H 17600 15200 50  0000 C CNN
-	1    17600 15200
-	1    0    0    -1
-$EndComp
-Wire Wire Line
-	17600 15350 17900 15350
-Connection ~ 18200 15350
-Connection ~ 17900 15350
-Wire Wire Line
-	17200 15050 17600 15050
-Connection ~ 18200 15050
-Connection ~ 17900 15050
-Connection ~ 17600 15050
-Text GLabel 18450 15350 2    39   Input ~ 0
-VSSD
-$Comp
 L Device:C C51
 U 1 1 599F4817
@@
 	24450 9800 24750 9800
 Wire Wire Line
-	25050 9700 25300 9700
-Wire Wire Line
-	24750 9700 25050 9700
-Wire Wire Line
-	25050 9400 25300 9400
-Wire Wire Line
-	24750 9400 25050 9400
-Wire Wire Line
-	24450 9400 24750 9400
-Wire Wire Line
 	25050 9300 25300 9300
 Wire Wire Line
@@
 	17850 9600 18150 9600
 Wire Wire Line
-	18450 9500 18700 9500
-Wire Wire Line
-	18150 9500 18450 9500
-Wire Wire Line
-	18450 9200 18700 9200
-Wire Wire Line
-	18150 9200 18450 9200
-Wire Wire Line
-	17850 9200 18150 9200
-Wire Wire Line
 	18450 9100 18700 9100
 Wire Wire Line
@@
 	24450 15500 24750 15500
 Wire Wire Line
-	25050 15400 25300 15400
-Wire Wire Line
-	24750 15400 25050 15400
-Wire Wire Line
-	25050 15100 25300 15100
-Wire Wire Line
-	24750 15100 25050 15100
-Wire Wire Line
-	24450 15100 24750 15100
-Wire Wire Line
 	25050 15000 25300 15000
 Wire Wire Line
@@
 Wire Wire Line
 	17600 15450 17900 15450
-Wire Wire Line
-	18200 15350 18450 15350
-Wire Wire Line
-	17900 15350 18200 15350
-Wire Wire Line
-	18200 15050 18450 15050
-Wire Wire Line
-	17900 15050 18200 15050
-Wire Wire Line
-	17600 15050 17900 15050
 Wire Wire Line
 	18200 14950 18450 14950
@@
 Wire Wire Line
 	20600 1400 19800 1400
+Wire Wire Line
+	17200 15050 18450 15050
+Wire Wire Line
+	24050 15100 25300 15100
+Wire Wire Line
+	24050 9400 25300 9400
+Wire Wire Line
+	17450 9200 18700 9200
 $EndSCHEMATC

Commit message: In Layout 2_19, heavily cleaned up routing from MUXes to the package to follow a standard pitch guideline. Cleaned up silkscreen. Renamed some SMD components to improve clarity.
Parts:
- renumbered R15 to RBT1, R16 to RBT2, R8 to RG1
Changed lines of the file:
@@
 $EndComp
 $Comp
-L Device:R R8
+L Device:R RG1
 U 1 1 599FAA80
 P 14550 1800
-F 0 "R8" V 14630 1800 50  0000 C CNN
+F 0 "RG1" V 14630 1800 50  0000 C CNN
 F 1 "1M" V 14550 1800 50  0000 C CNN
 F 2 "Resistor_SMD:R_0603_1608Metric" V 14480 1800 50  0001 C CNN
@@
 	17250 5150 17300 5150
 $Comp
-L Device:R R15
+L Device:R RBT1
 U 1 1 59A1B88E
 P 3350 1300
-F 0 "R15" V 3430 1300 50  0000 C CNN
+F 0 "RBT1" V 3430 1300 50  0000 C CNN
 F 1 "1k" V 3350 1300 50  0000 C CNN
 F 2 "Resistor_SMD:R_0603_1608Metric" V 3280 1300 50  0001 C CNN
@@
 $EndComp
 $Comp
-L Device:R R16
+L Device:R RBT2
 U 1 1 59A1BA2B
 P 3050 1300
-F 0 "R16" V 3130 1300 50  0000 C CNN
+F 0 "RBT2" V 3130 1300 50  0000 C CNN
 F 1 "2k" V 3050 1300 50  0000 C CNN
 F 2 "Resistor_SMD:R_0603_1608Metric" V 2980 1300 50  0001 C CNN

Commit message: Rotated bluetooth header connector on Layout 2_19
Changed lines of the file:
@@
 Wire Wire Line
 	17450 9200 18700 9200
+Text GLabel 3700 1550 2    39   Input ~ 0
+BT1_RXR
+Text GLabel 3700 1650 2    39   Input ~ 0
+BT1_TX
+Text GLabel 3700 1750 2    39   Input ~ 0
+GND
+Text GLabel 3700 1850 2    39   Input ~ 0
+VDDD
 $EndSCHEMATC
