File: PCB Layouts/Layout CHG1/Project.sch (KiCad schematic (older format))
At the start: 10 parts, among them J1 Conn_01x04

Commit message: Updated Lipo charger PCB to include changeover diode so that the battery can be used to power the circuit in the absence of an external power supply
Parts:
- added D1: D, Diode_SMD:D_0603_1608Metric, symbol Device:D
- D2: renamed from D1; value CRG -> CHG
- RREF1: value 2k -> 5k
- renumbered D2 to D3
Connections:
- net labels added: PROG, STAT
- wire segments 24 -> 26
Changed lines of the file:
@@
 EESchema Schematic File Version 4
-LIBS:Project-cache
 EELAYER 26 0
 EELAYER END
@@
 Connection ~ 3700 2250
 $Comp
-L Device:LED D1
+L Device:LED D2
 U 1 1 5E4B8767
 P 4000 3600
-F 0 "D1" V 4038 3483 50  0000 R CNN
-F 1 "CRG" V 3947 3483 50  0000 R CNN
+F 0 "D2" V 4038 3483 50  0000 R CNN
+F 1 "CHG" V 3947 3483 50  0000 R CNN
 F 2 "LED_SMD:LED_0603_1608Metric" H 4000 3600 50  0001 C CNN
 F 3 "~" H 4000 3600 50  0001 C CNN
@@
 	5300 4350 5300 2650
 $Comp
-L Device:LED D2
+L Device:LED D3
 U 1 1 5E4B9154
 P 4650 3600
-F 0 "D2" V 4595 3678 50  0000 L CNN
+F 0 "D3" V 4595 3678 50  0000 L CNN
 F 1 "DONE" V 4686 3678 50  0000 L CNN
 F 2 "LED_SMD:LED_0603_1608Metric" H 4650 3600 50  0001 C CNN
@@
 P 4300 2850
 F 0 "RREF1" H 4230 2804 50  0000 R CNN
-F 1 "2k" H 4230 2895 50  0000 R CNN
+F 1 "5k" H 4230 2895 50  0000 R CNN
 F 2 "Resistor_SMD:R_0603_1608Metric" V 4230 2850 50  0001 C CNN
 F 3 "~" H 4300 2850 50  0001 C CNN
@@
 	4000 4350 4650 4350
 Connection ~ 4650 4350
+Text GLabel 4300 2650 0    50   Input ~ 0
+PROG
+Text GLabel 5300 2650 2    50   Input ~ 0
+STAT
+$Comp
+L Device:D D1
+U 1 1 5E4BA0EB
+P 3700 2000
+F 0 "D1" V 3746 1921 50  0000 R CNN
+F 1 "D" V 3655 1921 50  0000 R CNN
+F 2 "Diode_SMD:D_0603_1608Metric" H 3700 2000 50  0001 C CNN
+F 3 "~" H 3700 2000 50  0001 C CNN
+	1    3700 2000
+	0    -1   -1   0
+$EndComp
+Text GLabel 3700 1750 1    50   Input ~ 0
+VBAT
+Wire Wire Line
+	3700 1750 3700 1850
+Wire Wire Line
+	3700 2150 3700 2250
 $EndSCHEMATC

Commit message: Added custom JST Lipo Header to Lipo Charging Layout
Parts:
- JSTPH1: footprint Connector_JST:JST_PH_S2B-PH-K_1x02_P2.00mm_Horizontal -> Custom_Footprint_Library:JST Lipo Header (S2B-PH-SM4-TB)
Changed lines of the file:
@@
 F 0 "JSTPH1" H 6380 2442 50  0000 L CNN
 F 1 "Conn_01x02" H 6380 2351 50  0000 L CNN
-F 2 "Connector_JST:JST_PH_S2B-PH-K_1x02_P2.00mm_Horizontal" H 6300 2450 50  0001 C CNN
+F 2 "Custom_Footprint_Library:JST Lipo Header (S2B-PH-SM4-TB)" H 6300 2450 50  0001 C CNN
 F 3 "~" H 6300 2450 50  0001 C CNN
 	1    6300 2450
