File: PCB Layouts/Layout CG2/Project.kicad_pcb (KiCad board)
At the start: 2 copper layers, 20 x 20 mm, 13 parts, among them J1 Conn_01x04

Commit message: Added new PCB layout for a combination BT and battery-powered board. Did initial placement of the 3.3V regulator, LEDs, and CMD jumper. Also fixed the RX/TX pinout for all of these accessory boards
Connections:
- J1 pad 3: RX -> TX
- J1 pad 4: TX -> RX
Changed lines of the file:
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@@
       (net 1 GND))
     (pad 3 thru_hole oval (at 0 5.08) (size 1.7 1.7) (drill 1) (layers *.Cu *.Mask)
+      (net 5 TX))
+    (pad 4 thru_hole oval (at 0 7.62) (size 1.7 1.7) (drill 1) (layers *.Cu *.Mask)
       (net 4 RX))
-    (pad 4 thru_hole oval (at 0 7.62) (size 1.7 1.7) (drill 1) (layers *.Cu *.Mask)
-      (net 5 TX))
     (model ${KISYS3DMOD}/Connector_PinHeader_2.54mm.3dshapes/PinHeader_1x04_P2.54mm_Vertical.wrl
       (at (xyz 0 0 0))
