File: PCB Layouts/Layout BT1/Project.sch (KiCad schematic (older format))
At the start: 22 parts, among them J1 Conn_01x04

Commit message: Made a custom footprint for the EGBT-045MS daughter board and added it to Layout BT1. The initial layout is now and complete and I just need to check over it for any mistakes or improvements.
Parts:
- removed D5: LED2_PAIRED, LED_SMD:LED_0603_1608Metric, symbol Device:LED
- removed R5: 1k, Resistor_SMD:R_0603_1608Metric, symbol Device:R
- added BTU1: EGBT-045MS, Custom_Footprint_Library:EGBT-045MS, symbol Custom_Schematic_Library:EGBT-045MS
Connections:
- net labels added: LED1, LED2
- wire segments 54 -> 60
Changed lines of the file:
@@
 L Device:LED D4
 U 1 1 5E69C45C
-P 9300 2900
-F 0 "D4" V 9338 2783 50  0000 R CNN
-F 1 "LED1_STATUS" V 9247 2783 50  0000 R CNN
-F 2 "LED_SMD:LED_0603_1608Metric" H 9300 2900 50  0001 C CNN
-F 3 "~" H 9300 2900 50  0001 C CNN
-	1    9300 2900
-	0    -1   -1   0
-$EndComp
-$Comp
-L Device:LED D5
-U 1 1 5E69C5F1
-P 10050 2900
-F 0 "D5" V 10088 2783 50  0000 R CNN
-F 1 "LED2_PAIRED" V 9997 2783 50  0000 R CNN
-F 2 "LED_SMD:LED_0603_1608Metric" H 10050 2900 50  0001 C CNN
-F 3 "~" H 10050 2900 50  0001 C CNN
-	1    10050 2900
+P 7550 3500
+F 0 "D4" V 7588 3383 50  0000 R CNN
+F 1 "LED1_STATUS" V 7497 3383 50  0000 R CNN
+F 2 "LED_SMD:LED_0603_1608Metric" H 7550 3500 50  0001 C CNN
+F 3 "~" H 7550 3500 50  0001 C CNN
+	1    7550 3500
 	0    -1   -1   0
 $EndComp
@@
 L Device:R R4
 U 1 1 5E69CA38
-P 9300 3400
-F 0 "R4" H 9230 3354 50  0000 R CNN
-F 1 "1k" H 9230 3445 50  0000 R CNN
-F 2 "Resistor_SMD:R_0603_1608Metric" V 9230 3400 50  0001 C CNN
-F 3 "~" H 9300 3400 50  0001 C CNN
-	1    9300 3400
-	-1   0    0    1
-$EndComp
-$Comp
-L Device:R R5
-U 1 1 5E69CBA8
-P 10050 3400
-F 0 "R5" H 9980 3354 50  0000 R CNN
-F 1 "1k" H 9980 3445 50  0000 R CNN
-F 2 "Resistor_SMD:R_0603_1608Metric" V 9980 3400 50  0001 C CNN
-F 3 "~" H 10050 3400 50  0001 C CNN
-	1    10050 3400
+P 7550 4000
+F 0 "R4" H 7480 3954 50  0000 R CNN
+F 1 "1k" H 7480 4045 50  0000 R CNN
+F 2 "Resistor_SMD:R_0603_1608Metric" V 7480 4000 50  0001 C CNN
+F 3 "~" H 7550 4000 50  0001 C CNN
+	1    7550 4000
 	-1   0    0    1
 $EndComp
 Wire Wire Line
-	9300 3050 9300 3250
-Wire Wire Line
-	10050 3050 10050 3250
-Text GLabel 9300 3750 3    50   Input ~ 0
-GND
-Text GLabel 10050 3750 3    50   Input ~ 0
+	7550 3650 7550 3850
+Text GLabel 7550 4350 3    50   Input ~ 0
 GND
 Wire Wire Line
-	10050 3550 10050 3750
-Wire Wire Line
-	9300 3550 9300 3750
+	7550 4150 7550 4350
 $Comp
 L Device:R R6
 U 1 1 5E6A6224
-P 10300 1350
-F 0 "R6" H 10230 1304 50  0000 R CNN
-F 1 "10k" H 10230 1395 50  0000 R CNN
-F 2 "Resistor_SMD:R_0603_1608Metric" V 10230 1350 50  0001 C CNN
-F 3 "~" H 10300 1350 50  0001 C CNN
-	1    10300 1350
+P 7550 2450
+F 0 "R6" H 7480 2404 50  0000 R CNN
+F 1 "10k" H 7480 2495 50  0000 R CNN
+F 2 "Resistor_SMD:R_0603_1608Metric" V 7480 2450 50  0001 C CNN
+F 3 "~" H 7550 2450 50  0001 C CNN
+	1    7550 2450
 	-1   0    0    1
 $EndComp
@@
 L Jumper:SolderJumper_2_Open JP1
 U 1 1 5E6A6FEF
-P 10450 1000
-F 0 "JP1" H 10450 1205 50  0000 C CNN
-F 1 "SolderJumper_2_Open" H 10450 1114 50  0000 C CNN
-F 2 "Jumper:SolderJumper-2_P1.3mm_Open_RoundedPad1.0x1.5mm" H 10450 1000 50  0001 C CNN
-F 3 "~" H 10450 1000 50  0001 C CNN
-	1    10450 1000
+P 8000 2800
+F 0 "JP1" H 8000 3005 50  0000 C CNN
+F 1 "SolderJumper_2_Open" H 8000 2914 50  0000 C CNN
+F 2 "Jumper:SolderJumper-2_P1.3mm_Open_RoundedPad1.0x1.5mm" H 8000 2800 50  0001 C CNN
+F 3 "~" H 8000 2800 50  0001 C CNN
+	1    8000 2800
 	1    0    0    -1
 $EndComp
 Wire Wire Line
-	10300 1000 10300 1200
-Text GLabel 10300 1700 3    50   Input ~ 0
+	7550 2600 7550 2800
+Text GLabel 7550 2100 1    50   Input ~ 0
 GND
 Wire Wire Line
-	10300 1500 10300 1700
-Text GLabel 10700 1000 2    50   Input ~ 0
+	7550 2100 7550 2300
+Text GLabel 8250 2800 2    50   Input ~ 0
 V3_3
 Wire Wire Line
-	10600 1000 10700 1000
+	8150 2800 8250 2800
 Wire Wire Line
-	9300 2750 9300 2600
+	7550 3350 7550 3200
+$Comp
+L Custom_Schematic_Library:EGBT-045MS BTU1
+U 1 1 5E69D27D
+P 7050 3000
+F 0 "BTU1" H 7050 3465 50  0000 C CNN
+F 1 "EGBT-045MS" H 7050 3374 50  0000 C CNN
+F 2 "Custom_Footprint_Library:EGBT-045MS" H 7050 2800 50  0001 C CNN
+F 3 "" H 7050 2800 50  0001 C CNN
+	1    7050 3000
+	1    0    0    -1
+$EndComp
+Text GLabel 6550 3100 0    50   Input ~ 0
+V3_3
 Wire Wire Line
-	10050 2750 10050 2600
+	6550 3100 6650 3100
+Text GLabel 6550 3200 0    50   Input ~ 0
+GND
 Wire Wire Line
-	10300 1000 10000 1000
-Connection ~ 10300 1000
+	6550 3200 6650 3200
+Text GLabel 6550 2800 0    50   Input ~ 0
+TX
+Wire Wire Line
+	6550 2800 6650 2800
+Text GLabel 6550 2900 0    50   Input ~ 0
+RX
+Wire Wire Line
+	6550 2900 6650 2900
+Wire Wire Line
+	7450 3200 7550 3200
+Wire Wire Line
+	7450 3100 8300 3100
+Text GLabel 7550 3200 2    50   Input ~ 0
+LED1
+Text GLabel 8300 3100 2    50   Input ~ 0
+LED2
+Wire Wire Line
+	7850 2800 7550 2800
+Wire Wire Line
+	7450 2800 7550 2800
+Connection ~ 7550 2800
+Text GLabel 7000 3650 3    50   Input ~ 0
+GND
+Text GLabel 7100 3650 3    50   Input ~ 0
+GND
+Wire Wire Line
+	7100 3550 7100 3650
+Wire Wire Line
+	7000 3550 7000 3650
 $EndSCHEMATC
