File: PCB Layouts/Layout RED3/Selection Interface.kicad_pcb (KiCad board)
At the start: 4 copper layers, 107.5 x 80 mm, 86 parts

Commit message: Updated Layout RED3 with the rearranged capacitor values (based on recommendation to place low value capacitors as close as possible to the IC since they can provide the fastest response time when the IC demands power)
Parts:
- C10, C19, C21, C42, C44, C9: value 47uF -> 0.1uF
- C13, C14, C33, C35, C51, C53: value 0.1uF -> 47uF
Changed lines of the file:
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@@
       (effects (font (size 1 1) (thickness 0.15)))
     )
-    (fp_text value 47uF (at -3.25 0) (layer F.Fab)
+    (fp_text value 0.1uF (at -3.25 0) (layer F.Fab)
       (effects (font (size 1 1) (thickness 0.15)))
     )
@@
       (effects (font (size 1 1) (thickness 0.15)))
     )
-    (fp_text value 47uF (at 0 0) (layer F.Fab)
+    (fp_text value 0.1uF (at 0 0) (layer F.Fab)
       (effects (font (size 1 1) (thickness 0.15)))
     )
@@
       (effects (font (size 1 1) (thickness 0.15)))
     )
-    (fp_text value 0.1uF (at -3.5 0) (layer F.Fab)
+    (fp_text value 47uF (at -3.5 0) (layer F.Fab)
       (effects (font (size 1 1) (thickness 0.15)))
     )
@@
       (effects (font (size 1 1) (thickness 0.15)))
     )
-    (fp_text value 0.1uF (at 0 0) (layer F.Fab)
+    (fp_text value 47uF (at 0 0) (layer F.Fab)
       (effects (font (size 1 1) (thickness 0.15)))
     )
@@
       (effects (font (size 1 1) (thickness 0.15)))
     )
-    (fp_text value 47uF (at 3.5 0.015 180) (layer F.Fab)
+    (fp_text value 0.1uF (at 3.5 0.015 180) (layer F.Fab)
       (effects (font (size 1 1) (thickness 0.15)))
     )
@@
       (effects (font (size 1 1) (thickness 0.15)))
     )
-    (fp_text value 47uF (at -4 0.015 180) (layer F.Fab)
+    (fp_text value 0.1uF (at -4 0.015 180) (layer F.Fab)
       (effects (font (size 1 1) (thickness 0.15)))
     )
@@
       (effects (font (size 1 1) (thickness 0.15)))
     )
-    (fp_text value 0.1uF (at 3.75 0.115 180) (layer F.Fab)
+    (fp_text value 47uF (at 3.75 0.115 180) (layer F.Fab)
       (effects (font (size 1 1) (thickness 0.15)))
     )
@@
       (effects (font (size 1 1) (thickness 0.15)))
     )
-    (fp_text value 0.1uF (at -3.75 0.115 180) (layer F.Fab)
+    (fp_text value 47uF (at -3.75 0.115 180) (layer F.Fab)
       (effects (font (size 1 1) (thickness 0.15)))
     )
@@
       (effects (font (size 1 1) (thickness 0.15)))
     )
-    (fp_text value 47uF (at -3.5 -0.115) (layer F.Fab)
+    (fp_text value 0.1uF (at -3.5 -0.115) (layer F.Fab)
       (effects (font (size 1 1) (thickness 0.15)))
     )
@@
       (effects (font (size 1 1) (thickness 0.15)))
     )
-    (fp_text value 47uF (at 4 -0.115) (layer F.Fab)
+    (fp_text value 0.1uF (at 4 -0.115) (layer F.Fab)
       (effects (font (size 1 1) (thickness 0.15)))
     )
@@
       (effects (font (size 1 1) (thickness 0.15)))
     )
-    (fp_text value 0.1uF (at -3.75 -0.015) (layer F.Fab)
+    (fp_text value 47uF (at -3.75 -0.015) (layer F.Fab)
       (effects (font (size 1 1) (thickness 0.15)))
     )
@@
       (effects (font (size 1 1) (thickness 0.15)))
     )
-    (fp_text value 0.1uF (at 3.75 0) (layer F.Fab)
+    (fp_text value 47uF (at 3.75 0) (layer F.Fab)
       (effects (font (size 1 1) (thickness 0.15)))
     )
@@
       (effects (font (size 1 1) (thickness 0.15)))
     )
-    (fp_text value 1uF (at -3 0 270) (layer F.Fab)
+    (fp_text value 1uF (at 0 -1.4 270) (layer F.Fab)
       (effects (font (size 1 1) (thickness 0.15)))
     )
